File: perovskite_switcher/Perovskite_Switches.sch (KiCad schematic (older format))
At the start: 45 parts, among them J1 G125-MV12605M1P, Q1 DMC2053UVT, U1 SN74LVC1G14DRL, U10 MAX4736EUBT, U11 MAX4736EUBT, U12 MAX4736EUBT, U13 MAX4736EUBT, U14 MAX4736EUBT, U15 LT3092ETS8TRPBF, U16 INA180B2IDBVT, U17 MCP6401RT-xOT, U2 CD4518BM96, U3 CD4028BMT, U4 CD4028BMT, U5 MAX4736EUBT, U6 MAX4736EUBT, U7 MAX4736EUBT, U8 MAX4736EUBT, U9 MAX4736EUBT

Commit message: Update boards
- Added flight computer board outline
- Added GUI for curve tracer
- Updated curve tracer
- Updated perovskite switcher
Parts:
- added C? (x7): 0.1u, symbol Device:C
Connections:
- net +3V3: now also C?.1, C?.1, C?.1, C?.1, C?.1, C?.1
- net GND: now also J1.14, J1.15, J1.16, J1.17, J1.18, J1.19, J1.20, J1.23, C?.1, C?.2, C?.2, C?.2, C?.2, C?.2, C?.2
- net at U14.10 (COM1): no longer J1.14
- net at U13.6 (COM2): now also J1.22; no longer J1.15
- net at U13.10 (COM1): now also J1.21; no longer J1.16
- net at U12.6 (COM2): now also J1.24; no longer J1.17
- net at U12.10 (COM1): now also J1.25; no longer J1.18
- net at U11.6 (COM2): now also J1.26; no longer J1.19
- net at Q1.4 (D), U15.7 (IN_2), U15.8 (IN): now also C?.2
Other:
- moved on the sheet: U17
