File: perovskite_switcher/switcher.sch (KiCad schematic (older format))
At the start: 0 parts

Commit message: Update boards
- Added flight computer board outline
- Added GUI for curve tracer
- Updated curve tracer
- Updated perovskite switcher
Parts:
- added C1, C10, C11, C12, C14, C16, C18, C2, C20, C22, C24, C26, C4, C6, C8: 0.1u, Capacitor_SMD:C_0603_1608Metric, symbol Device:C
- added FB1: Ferrite_Bead, Inductor_SMD:L_0603_1608Metric, symbol Device:Ferrite_Bead
- added J1, J2: Conn_01x10_Female, Connector_PinHeader_2.54mm:PinHeader_1x10_P2.54mm_Vertical, symbol Connector:Conn_01x10_Female
- added J3: G125-MV12605M1P, LIB_G125-MV12605M1P:G125-MV12605M1P, symbol G125-MV12605M1P:G125-MV12605M1P
- added J4: Panel Output to Curve Tracer, Connector_PinHeader_2.54mm:PinHeader_1x01_P2.54mm_Vertical, symbol Connector:Conn_01x01_Female
- added J5: Silicon Cell, Connector_PinHeader_2.54mm:PinHeader_1x02_P2.54mm_Vertical, symbol Connector:Conn_01x02_Female
- added Q1: DMC2053UVT, Package_TO_SOT_SMD:TSOT-23-6, symbol Transistor_FET:DMC2053UVT
- added R1: 1k, Resistor_SMD:R_0603_1608Metric, symbol Device:R
- added R10, R11, R12, R13, R14, R15, R16, R17, R18, R19, R20, R21, R22, R23, R4, R5, R6, R7, R8, R9: R, Resistor_SMD:R_0603_1608Metric, symbol Device:R
- added R2, R3: 10k, Resistor_SMD:R_0603_1608Metric, symbol Device:R
- added R24: 20k, Resistor_SMD:R_0603_1608Metric, symbol Device:R
- added R25, R27, R28, R29, R30: 100, Resistor_SMD:R_0603_1608Metric, symbol Device:R
- added R26: 1, Resistor_SMD:R_0603_1608Metric, symbol Device:R
- added U1: SN74LVC1G14DRL, Package_TO_SOT_SMD:SOT-23-5, symbol 74xGxx:SN74LVC1G14DRL
- added U10, U11, U12, U13, U14, U5, U6, U7, U8, U9: MAX4736EUBT, MAX4736EUBT:SOP50P490X110-10N, symbol MAX4736EUBT:MAX4736EUBT
- added U15: LT3092ETS8TRPBF, LT3092ETS8TRPBF:TSOT-23_TS8, symbol LT3092ETS8TRPBF:LT3092ETS8TRPBF
- added U2: CD4518BM96, ul_CD4518BM96:CD4518BM96, symbol CD4518BM96:CD4518BM96
- added U3, U4: CD4028BMT, CD4028BMT:SOIC127P600X175-16N, symbol CD4028BMT:CD4028BMT
Connections:
- new net: J2.4 (Pin_4), R25.2
- new net: J4.1 (Pin_1), U10.2 (NO1), U10.4 (NO2), U11.2 (NO1), U11.4 (NO2), U12.2 (NO1), U12.4 (NO2), U13.2 (NO1), U13.4 (NO2), U14.2 (NO1), U14.4 (NO2), U5.2 (NO1), U5.4 (NO2), U6.2 (NO1), U6.4 (NO2), U7.2 (NO1), U7.4 (NO2), U8.2 (NO1), U8.4 (NO2), U9.2 (NO1), U9.4 (NO2)
- new net: J5.1 (Pin_1), U14.10 (COM1)
- new net: J2.2 (Pin_2), R27.2
- new net: J2.3 (Pin_3), R28.2
- new net: J1.5 (Pin_5), R29.2
- new net: J1.6 (Pin_6), R30.1
- new net: FB1.2, J1.1 (Pin_1)
- new net: U3.14 (1), U5.1 (IN1)
- new net: J3.7, U5.10 (COM1)
- new net: U3.15 (3), U5.5 (IN2)
- new net: J3.8, U5.6 (COM2)
- new net: R5.2, U5.7 (NC2)
- new net: R4.2, U5.9 (NC1)
- new net: U3.2, U6.1 (IN1)
- new net: J3.5, U6.10 (COM1)
- new net: U3.1 (4), U6.5 (IN2)
- new net: J3.6, U6.6 (COM2)
- new net: R7.2, U6.7 (NC2)
- new net: R6.2, U6.9 (NC1)
- new net: U3.4 (7), U7.1 (IN1)
- new net: J3.3, U7.10 (COM1)
- new net: U3.3 (0), U7.5 (IN2)
- new net: J3.4, U7.6 (COM2)
- new net: R9.2, U7.7 (NC2)
- new net: R8.2, U7.9 (NC1)
- new net: U3.6 (5), U8.1 (IN1)
- new net: J3.1, U8.10 (COM1)
- new net: U3.5 (9), U8.5 (IN2)
- new net: J3.2, U8.6 (COM2)
- new net: R11.2, U8.7 (NC2)
- new net: R10.2, U8.9 (NC1)
- new net: U3.9 (8), U9.1 (IN1)
- new net: J3.22, U9.10 (COM1)
- new net: U3.7 (6), U9.5 (IN2)
- new net: J3.21, U9.6 (COM2)
- new net: R13.2, U9.7 (NC2)
- new net: R12.2, U9.9 (NC1)
- new net: U10.1 (IN1), U4.14 (1)
- new net: J3.25, U10.10 (COM1)
- new net: U10.5 (IN2), U4.15 (3)
- new net: J3.24, U10.6 (COM2)
- new net: R15.2, U10.7 (NC2)
- new net: R14.2, U10.9 (NC1)
- new net: U11.1 (IN1), U4.2
- new net: J3.13, U11.10 (COM1)
- new net: U11.5 (IN2), U4.1 (4)
- new net: J3.26, U11.6 (COM2)
- new net: R17.2, U11.7 (NC2)
- new net: R16.2, U11.9 (NC1)
- new net: U12.1 (IN1), U4.4 (7)
- new net: J3.11, U12.10 (COM1)
- new net: U12.5 (IN2), U4.3 (0)
- new net: J3.12, U12.6 (COM2)
- new net: R19.2, U12.7 (NC2)
- new net: R18.2, U12.9 (NC1)
- new net: U13.1 (IN1), U4.6 (5)
- new net: J3.9, U13.10 (COM1)
- new net: U13.5 (IN2), U4.5 (9)
- new net: J3.10, U13.6 (COM2)
- new net: R21.2, U13.7 (NC2)
- new net: R20.2, U13.9 (NC1)
- new net: U14.1 (IN1), U4.9 (8)
- new net: U14.5 (IN2), U4.7 (6)
- new net: R24.1, R26.1, U14.6 (COM2)
- new net: R23.2, U14.7 (NC2)
- new net: R22.2, U14.9 (NC1)
- new net: U2.11 (Q1B), U3.10 (A)
- new net: U2.12 (Q2B), U3.13 (B)
- new net: U2.13 (Q3B), U3.12 (C)
- new net: U2.14 (Q4B), U3.11 (D)
- new net: U1.4, U2.2 (ENABLEA)
- new net: U2.3 (Q1A), U4.10 (A)
- new net: U2.4 (Q2A), U4.13 (B)
- new net: U2.5 (Q3A), U4.12 (C)
- new net: U2.6 (Q4A), U4.11 (D)
- new net: Q1.1 (G), R1.1, R2.1
- new net: Q1.3 (G), Q1.6 (D), R3.2
- new net: C26.2, Q1.4 (D), U15.7 (IN_2), U15.8 (IN)
- new net: R26.2, U15.2 (OUT_2), U15.3 (OUT_3), U15.4 (OUT)
- new net: R24.2, U15.5 (SET)
- new net +3V3: C1.1, C10.1, C11.1, C12.1, C14.1, C16.1, C18.1, C2.1, C20.1, C22.1, C24.1, C4.1, C6.1, C8.1, FB1.1, Q1.2 (S), R3.1, U1.5 (VCC), U10.8 (V+), U11.8 (V+), U12.8 (V+), U13.8 (V+), U14.8 (V+), U2.16 (VDD), U3.16 (VDD), U4.16 (VDD), U5.8 (V+), U6.8 (V+), U7.8 (V+), U8.8 (V+), U9.8 (V+)
- new net 0-9_CLOCK: R25.1, U2.1 (CLOCKA)
- new net 10-19_CLOCK: R28.1, U2.9 (CLOCKB)
- new net ENABLE_PANEL_SWITCH: R27.1, U1.2, U2.10 (ENABLEB)
- new net ENABLE_TEST_SOURCE: R1.2, R29.1
- new net GND: C1.2, C10.2, C11.2, C12.2, C14.2, C16.2, C18.2, C2.2, C20.2, C22.2, C24.2, C26.1, C4.2, C6.2, C8.2, J2.10 (Pin_10), J3.14, J3.15, J3.16, J3.17, J3.18, J3.19, J3.20, J3.23, J5.2 (Pin_2), Q1.5 (S), R10.1, R11.1, R12.1, R13.1, R14.1, R15.1, R16.1, R17.1, R18.1, R19.1, R2.2, R20.1, R21.1, R22.1, R23.1, R4.1, R5.1, R6.1, R7.1, R8.1, R9.1, U1.3 (GND), U10.3 (GND), U11.3 (GND), U12.3 (GND), U13.3 (GND), U14.3 (GND), U2.8 (VSS), U3.8 (VSS), U4.8 (VSS), U5.3 (GND), U6.3 (GND), U7.3 (GND), U8.3 (GND), U9.3 (GND)
- new net RESET_PANEL_SWITCH: R30.2, U2.15 (RESETB), U2.7 (RESETA)
