File: resistor_ladder_curve_tracer/resistor_ladder.sch (KiCad schematic (older format))
At the start: 26 parts, among them U10 ADG841YKSZ-500RL7, U11 ADG841YKSZ-500RL7, U12 ADG841YKSZ-500RL7, U13 ADG841YKSZ-500RL7, U5 74HC590, U6 ADG841YKSZ-500RL7, U7 ADG841YKSZ-500RL7, U8 ADG841YKSZ-500RL7, U9 ADG841YKSZ-500RL7

Commit message: Update boards
- Added flight computer board outline
- Added GUI for curve tracer
- Updated curve tracer
- Updated perovskite switcher
Connections:
- net LADDER_LATCH: now reaches U5.13 (CPR)
- no-connect marks 2 -> 1
Changed lines of the file:
@@
 Wire Wire Line
 	2500 5550 2600 5550
-NoConn ~ 2600 5150
 $Comp
 L Device:C C8
@@
 Wire Wire Line
 	3900 2050 3900 2350
+Wire Wire Line
+	2600 5150 2300 5150
+Text HLabel 2300 5150 0    50   Input ~ 0
+LADDER_LATCH
 $EndSCHEMATC

Commit message: Working on flight computer
- Update resistor ladder curve tracer silkscreen, schematic, and layout
- Flight computer schematic drafted for MSP430 circuits, updated curve tracer, perovskite switching network.
Changed lines of the file:
@@
 Sheet 2 3
 Title "Resistor 8-Bit Ladder"
-Date "2022-09-18"
-Rev "A"
+Date "2022-11-08"
+Rev "B"
 Comp "Advanced eXperimental Payloads | UNL Aerospace Club"
 Comment1 "Copyright (c) 2022"
@@
 L power:+3V3 #PWR0123
 U 1 1 63117816
-P 3700 2750
-F 0 "#PWR0123" H 3700 2600 50  0001 C CNN
-F 1 "+3V3" H 3715 2923 50  0000 C CNN
-F 2 "" H 3700 2750 50  0001 C CNN
-F 3 "" H 3700 2750 50  0001 C CNN
-	1    3700 2750
+P 3900 3050
+F 0 "#PWR0123" H 3900 2900 50  0001 C CNN
+F 1 "+3V3" H 3915 3223 50  0000 C CNN
+F 2 "" H 3900 3050 50  0001 C CNN
+F 3 "" H 3900 3050 50  0001 C CNN
+	1    3900 3050
 	1    0    0    -1
 $EndComp
@@
 	5150 2050 5800 2050
 Wire Wire Line
-	3700 3350 3700 2750
-Wire Wire Line
 	4300 3250 4300 3350
-Connection ~ 4300 3350
-Wire Wire Line
-	4300 3350 3700 3350
 Wire Wire Line
 	4950 3250 4950 3350
@@
 Text HLabel 2300 5150 0    50   Input ~ 0
 LADDER_LATCH
+Wire Wire Line
+	4300 3350 3900 3350
+Wire Wire Line
+	3900 3350 3900 3050
+Connection ~ 4300 3350
 $EndSCHEMATC
