File: flight_computer/sat_comms.sch (KiCad schematic (older format))
At the start: 0 parts

Commit message: Updating flight computer
- Added datasheets for peripherals
- Added resistor ladder firmware
- Added perovskite switcher firmware
- Started flight computer firmware
- Added curve comparisons
- Updating flight computer schematic
Parts:
- added J?: EyeStar, symbol Connector:Conn_01x04_Male
Connections:
- new net BUSY_IN: J?.2 (Pin_2)
- new net GND: J?.1 (Pin_1)
- new net RX_IN: J?.4 (Pin_4)
- new net TX_OUT: J?.3 (Pin_3)
Changed lines of the file:
@@
 $Descr A4 11693 8268
 encoding utf-8
-Sheet 1 9
+Sheet 9 9
 Title ""
 Date ""
@@
 Comment4 ""
 $EndDescr
+$Comp
+L Connector:Conn_01x04_Male J?
+U 1 1 637A3118
+P 6050 3600
+F 0 "J?" H 6022 3482 50  0000 R CNN
+F 1 "EyeStar" H 6022 3573 50  0000 R CNN
+F 2 "" H 6050 3600 50  0001 C CNN
+F 3 "~" H 6050 3600 50  0001 C CNN
+	1    6050 3600
+	-1   0    0    1
+$EndComp
+$Comp
+L power:GND #PWR?
+U 1 1 637A3C71
+P 5850 3700
+F 0 "#PWR?" H 5850 3450 50  0001 C CNN
+F 1 "GND" H 5855 3527 50  0000 C CNN
+F 2 "" H 5850 3700 50  0001 C CNN
+F 3 "" H 5850 3700 50  0001 C CNN
+	1    5850 3700
+	1    0    0    -1
+$EndComp
+Text HLabel 5850 3400 0    50   Output ~ 0
+RX_IN
+Text HLabel 5850 3500 0    50   Input ~ 0
+TX_OUT
+Text HLabel 5850 3600 0    50   Output ~ 0
+BUSY_IN
 $EndSCHEMATC
