File: flight_computer/flight_computer.kicad_pcb (KiCad board)
At the start: 2 copper layers, 87 x 75 mm, 0 parts

Commit message: Continuing layout
Parts:
- added C1: 0.1u, Capacitor_SMD:C_0603_1608Metric, F.Cu at (200.5, 37.4)
- added C10: 0.1u, Capacitor_SMD:C_0603_1608Metric, F.Cu at (97.3, 49.5)
- added C11: 0.1u, Capacitor_SMD:C_0603_1608Metric, F.Cu at (160.7, 163.6)
- added C16: 0.1u, Capacitor_SMD:C_0603_1608Metric, F.Cu at (164.4, 165.6)
- added C18: 220n, Capacitor_SMD:C_0603_1608Metric, F.Cu at (137.5, 171.3)
- added C2: 0.1u, Capacitor_SMD:C_0603_1608Metric, F.Cu at (200.5, 46.4)
- added C20: 1u, Capacitor_SMD:C_0603_1608Metric, F.Cu at (159.9, 172.1)
- added C21: 10n, Capacitor_SMD:C_0603_1608Metric, F.Cu at (150.0, 172.7)
- added C22: 10n, Capacitor_SMD:C_0603_1608Metric, F.Cu at (152.3, 170.2)
- added C23: 10n, Capacitor_SMD:C_0603_1608Metric, F.Cu at (150.0, 165.3)
- added C24: 10n, Capacitor_SMD:C_0603_1608Metric, F.Cu at (152.3, 167.8)
- added C25: 10u, Capacitor_SMD:C_0603_1608Metric, F.Cu at (155.4, 175.2)
- added C26: 10u, Capacitor_SMD:C_0603_1608Metric, F.Cu at (155.4, 164.5)
- added C27: 0.1u, Capacitor_SMD:C_0603_1608Metric, F.Cu at (150.4, 45.5)
- added C28: 0.1u, Capacitor_SMD:C_0603_1608Metric, F.Cu at (134.4, 45.5)
- added C29: 0.1u, Capacitor_SMD:C_0603_1608Metric, F.Cu at (139.8, 45.5)
- added C3: 0.1u, Capacitor_SMD:C_0603_1608Metric, F.Cu at (200.5, 55.4)
- added C30: 0.1u, Capacitor_SMD:C_0603_1608Metric, F.Cu at (123.7, 45.5)
- added C31: 0.1u, Capacitor_SMD:C_0603_1608Metric, F.Cu at (145.1, 45.5)
- added C32: 0.1u, Capacitor_SMD:C_0603_1608Metric, F.Cu at (166.4, 45.5)
- added C33: 0.1u, Capacitor_SMD:C_0603_1608Metric, F.Cu at (161.1, 45.5)
- added C34: 0.1u, Capacitor_SMD:C_0603_1608Metric, F.Cu at (129.1, 45.5)
- added C35: 0.1u, Capacitor_SMD:C_0603_1608Metric, F.Cu at (155.8, 45.5)
- added C36: 0.1u, Capacitor_SMD:C_0603_1608Metric, F.Cu at (171.8, 45.5)
- added C37: 0.1u, Capacitor_SMD:C_0603_1608Metric, F.Cu at (84.8, 61.3)
- added C38: 0.1u, Capacitor_SMD:C_0603_1608Metric, F.Cu at (75.8, 67.0)
- added C39: 0.1u, Capacitor_SMD:C_0603_1608Metric, F.Cu at (76.4, 49.1)
- added C4: 0.1u, Capacitor_SMD:C_0603_1608Metric, F.Cu at (200.5, 64.5)
- added C40: 0.1u, Capacitor_SMD:C_0603_1608Metric, F.Cu at (68.0, 48.9)
- added C41: 0.1u, Capacitor_SMD:C_0603_1608Metric, F.Cu at (108.8, 40.4)
- added C42: 0.1u, Capacitor_SMD:C_0603_1608Metric, F.Cu at (143.4, 174.1)
- added C43: 1u, Capacitor_SMD:C_0603_1608Metric, F.Cu at (159.9, 166.9)
- added C44: 10u, Capacitor_SMD:C_0603_1608Metric, F.Cu at (121.3, 94.9)
- added C45: 0.1u, Capacitor_SMD:C_0603_1608Metric, F.Cu at (121.3, 93.2)
- added C46: 0.1u, Capacitor_SMD:C_0603_1608Metric, F.Cu at (177.1, 45.5)
- added C5: 0.1u, Capacitor_SMD:C_0603_1608Metric, F.Cu at (200.5, 41.9)
- added C50: 0.1u, Capacitor_SMD:C_0603_1608Metric, F.Cu at (63.2, 104.3)
- added C52: 10u, Capacitor_SMD:C_0603_1608Metric, F.Cu at (141.5, 161.0)
- added C53: 0.1u, Capacitor_SMD:C_0603_1608Metric, F.Cu at (146.5, 156.7)
- added C54: 0.1u, Capacitor_SMD:C_0603_1608Metric, F.Cu at (151.4, 160.4)
- added C55: CP, Capacitor_SMD:C_0603_1608Metric, F.Cu at (153.0, 160.4)
- added C56: 0.1u, Capacitor_SMD:C_0603_1608Metric, F.Cu at (66.9, 91.1)
- added C57: 1u, Capacitor_SMD:C_0603_1608Metric, F.Cu at (65.3, 91.1)
- added C58: 10p, Capacitor_SMD:C_0603_1608Metric, F.Cu at (60.8, 88.8)
- added C59: 10p, Capacitor_SMD:C_0603_1608Metric, F.Cu at (62.3, 88.8)
- added C6: 0.1u, Capacitor_SMD:C_0603_1608Metric, F.Cu at (200.5, 50.9)
- added C60: 0.1u, Capacitor_SMD:C_0603_1608Metric, F.Cu at (55.8, 91.1)
- added C61: 0.1u, Capacitor_SMD:C_0603_1608Metric, F.Cu at (59.0, 91.1)
- added C62: 0.1u, Capacitor_SMD:C_0603_1608Metric, F.Cu at (183.1, 130.4)
- added C7: 0.1u, Capacitor_SMD:C_0603_1608Metric, F.Cu at (200.5, 59.9)
- added C8: 0.1u, Capacitor_SMD:C_0603_1608Metric, F.Cu at (200.5, 69.0)
- added FB2: Ferrite_Bead_Small, Inductor_SMD:L_0603_1608Metric, F.Cu at (57.4, 91.1)
- added J1: Silicon Cell, Connector_PinHeader_2.54mm:PinHeader_1x02_P2.54mm_Vertical, F.Cu at (173.0, 32.6)
- added J2: G125-MV12605M1P, LIB_G125-MV12605M1P:G125-MV12605M1P, F.Cu at (188.3, 111.4)
- added J3: Conn_01x08_Female, Connector_PinSocket_2.54mm:PinSocket_1x08_P2.54mm_Vertical, F.Cu at (117.6, 111.0)
- added J4: Conn_02x07_Odd_Even, Connector_PinSocket_2.54mm:PinSocket_2x08_P2.54mm_Vertical, F.Cu at (81.7, 117.0)
- added J5: 0781710004, 0781710004:MOLEX_0781710004, F.Cu at (185.4, 129.0)
- added Q1: DMC2053UVT, Package_TO_SOT_SMD:TSOT-23-6, F.Cu at (105.6, 40.2)
- added R1: 4.7k, Resistor_SMD:R_0603_1608Metric, F.Cu at (69.7, 99.6)
- added R10: 16000, Resistor_SMD:R_0603_1608Metric, F.Cu at (204.3, 35.5)
- added R11: 100k, Resistor_SMD:R_0603_1608Metric, F.Cu at (155.4, 158.1)
- added R12: 1k, Resistor_SMD:R_0603_1608Metric, F.Cu at (153.5, 152.6)
- added R13: 500k, Resistor_SMD:R_0603_1608Metric, F.Cu at (155.4, 161.2)
- added R14: 100k, Resistor_SMD:R_0603_1608Metric, F.Cu at (155.4, 159.6)
- added R15: 10k, Resistor_SMD:R_0603_1608Metric, F.Cu at (137.5, 168.1)
- added R16: 10k, Resistor_SMD:R_0603_1608Metric, F.Cu at (137.5, 169.7)
- added R17: 10k, Resistor_SMD:R_0603_1608Metric, F.Cu at (137.5, 166.5)
- added R18: 470, Resistor_SMD:R_0603_1608Metric, F.Cu at (152.3, 173.5)
- added R19: 470, Resistor_SMD:R_0603_1608Metric, F.Cu at (152.3, 171.9)
- added R2: 4.7k, Resistor_SMD:R_0603_1608Metric, F.Cu at (69.7, 98.0)
- added R20: 470, Resistor_SMD:R_0603_1608Metric, F.Cu at (152.3, 164.5)
- added R21: 470, Resistor_SMD:R_0603_1608Metric, F.Cu at (152.3, 166.1)
- added R22: 10k, Resistor_SMD:R_0603_1608Metric, F.Cu at (155.4, 173.5)
- added R23: 10k, Resistor_SMD:R_0603_1608Metric, F.Cu at (155.4, 162.8)
- added R24: 510m, Resistor_SMD:R_1206_3216Metric, F.Cu at (168.7, 167.6)
- added R25: 470, Resistor_SMD:R_0603_1608Metric, F.Cu at (164.8, 162.8)
- added R26: 10M, Resistor_SMD:R_0603_1608Metric, F.Cu at (167.9, 161.2)
- added R27: 10M, Resistor_SMD:R_0603_1608Metric, F.Cu at (164.8, 161.2)
- added R28: 1k, Resistor_SMD:R_0603_1608Metric, F.Cu at (100.6, 40.2)
- added R29: 10k, Resistor_SMD:R_0603_1608Metric, F.Cu at (102.2, 40.2)
- added R3: 50, Resistor_SMD:R_0603_1608Metric, F.Cu at (204.3, 67.1)
- added R30: 10k, Resistor_SMD:R_0603_1608Metric, F.Cu at (105.7, 37.7)
- added R31: R, Resistor_SMD:R_0603_1608Metric, F.Cu at (125.6, 40.5)
- added R32: R, Resistor_SMD:R_0603_1608Metric, F.Cu at (127.3, 40.5)
- added R33: R, Resistor_SMD:R_0603_1608Metric, F.Cu at (130.9, 40.5)
- added R34: R, Resistor_SMD:R_0603_1608Metric, F.Cu at (132.6, 40.5)
- added R35: R, Resistor_SMD:R_0603_1608Metric, F.Cu at (136.3, 40.5)
- added R36: R, Resistor_SMD:R_0603_1608Metric, F.Cu at (137.9, 40.5)
- added R37: R, Resistor_SMD:R_0603_1608Metric, F.Cu at (141.6, 40.5)
- added R38: R, Resistor_SMD:R_0603_1608Metric, F.Cu at (143.3, 40.5)
- added R39: R, Resistor_SMD:R_0603_1608Metric, F.Cu at (146.9, 40.5)
- added R4: 250, Resistor_SMD:R_0603_1608Metric, F.Cu at (204.3, 62.5)
- added R40: R, Resistor_SMD:R_0603_1608Metric, F.Cu at (148.6, 40.5)
- added R41: R, Resistor_SMD:R_0603_1608Metric, F.Cu at (152.3, 40.5)
- added R42: R, Resistor_SMD:R_0603_1608Metric, F.Cu at (153.9, 40.5)
- added R43: R, Resistor_SMD:R_0603_1608Metric, F.Cu at (157.5, 40.5)
- added R44: R, Resistor_SMD:R_0603_1608Metric, F.Cu at (159.2, 40.5)
- added R45: R, Resistor_SMD:R_0603_1608Metric, F.Cu at (162.9, 40.5)
- added R46: R, Resistor_SMD:R_0603_1608Metric, F.Cu at (164.5, 40.5)
- added R47: R, Resistor_SMD:R_0603_1608Metric, F.Cu at (168.3, 40.5)
- added R48: R, Resistor_SMD:R_0603_1608Metric, F.Cu at (169.9, 40.5)
- added R49: R, Resistor_SMD:R_0603_1608Metric, F.Cu at (173.6, 40.5)
- added R5: 500, Resistor_SMD:R_0603_1608Metric, F.Cu at (204.3, 58.0)
- added R50: R, Resistor_SMD:R_0603_1608Metric, F.Cu at (175.3, 40.5)
- added R51: 20k, Resistor_SMD:R_0603_1608Metric, F.Cu at (116.5, 39.6)
- added R52: 1, Resistor_SMD:R_0603_1608Metric, F.Cu at (116.5, 41.1)
- added R57: R, Resistor_SMD:R_0603_1608Metric, F.Cu at (64.8, 104.3)
- added R6: 1000, Resistor_SMD:R_0603_1608Metric, F.Cu at (204.3, 53.5)
- added R7: 2000, Resistor_SMD:R_0603_1608Metric, F.Cu at (204.3, 49.0)
- added R8: 4000, Resistor_SMD:R_0603_1608Metric, F.Cu at (204.3, 44.5)
- added R9: 8000, Resistor_SMD:R_0603_1608Metric, F.Cu at (204.3, 40.0)
- added SW2: SW_SPDT, Button_Switch_SMD:SW_SPDT_PCM12, F.Cu at (74.5, 119.3)
- added U1: 74HC590, Package_SO:SOIC-16_3.9x9.9mm_P1.27mm, F.Cu at (97.5, 55.6)
- added U10: OPA2387, Package_SON:WSON-8-1EP_2x2mm_P0.5mm_EP0.9x1.6mm, F.Cu at (160.7, 161.0)
- added U11: MCP4725xxx-xCH, Package_TO_SOT_SMD:SOT-23-6, F.Cu at (153.5, 155.3)
- added U12: ADS131M04IPWR, ADS131M04IPWR:SOP65P640X120-20N, F.Cu at (143.4, 169.4)
- added U13: INA190A4IDDFR, ul_INA190A4IDDFR:INA190A4IDDFR, F.Cu at (164.4, 168.2)
- added U15: SN74LVC1G14DRL, Package_TO_SOT_SMD:SOT-23-5, F.Cu at (76.1, 63.8)
- added U16: CD4518BM96, ul_CD4518BM96:CD4518BM96, F.Cu at (68.1, 55.4)
- added U17: CD4028BMT, CD4028BMT:SOIC127P600X175-16N, F.Cu at (76.5, 55.4)
- added U18: CD4028BMT, CD4028BMT:SOIC127P600X175-16N, F.Cu at (84.8, 55.4)
- added U19: MAX4736EUBT, MAX4736EUBT:SOP50P490X110-10N, F.Cu at (179.8, 45.5)
- added U2: ADG841YKSZ-500RL7, ul_ADG841YKSZ-500RL7:ADG841YKSZ-500RL7, F.Cu at (200.5, 66.8)
- added U20: MAX4736EUBT, MAX4736EUBT:SOP50P490X110-10N, F.Cu at (126.4, 45.5)
- added U21: MAX4736EUBT, MAX4736EUBT:SOP50P490X110-10N, F.Cu at (131.8, 45.5)
- added U22: MAX4736EUBT, MAX4736EUBT:SOP50P490X110-10N, F.Cu at (137.1, 45.5)
- added U23: MAX4736EUBT, MAX4736EUBT:SOP50P490X110-10N, F.Cu at (142.4, 45.5)
- added U24: MAX4736EUBT, MAX4736EUBT:SOP50P490X110-10N, F.Cu at (147.8, 45.5)
- added U25: MAX4736EUBT, MAX4736EUBT:SOP50P490X110-10N, F.Cu at (153.1, 45.5)
- added U26: MAX4736EUBT, MAX4736EUBT:SOP50P490X110-10N, F.Cu at (158.4, 45.5)
- added U27: MAX4736EUBT, MAX4736EUBT:SOP50P490X110-10N, F.Cu at (163.8, 45.5)
- added U28: MAX4736EUBT, MAX4736EUBT:SOP50P490X110-10N, F.Cu at (169.1, 45.5)
- added U29: MAX4736EUBT, MAX4736EUBT:SOP50P490X110-10N, F.Cu at (174.4, 45.5)
- added U3: ADG841YKSZ-500RL7, ul_ADG841YKSZ-500RL7:ADG841YKSZ-500RL7, F.Cu at (200.5, 62.2)
- added U30: LT3092EDD#TRPBF, LT3092EDD_TRPBF:DFN-8_DD, F.Cu at (111.9, 40.4)
- added U31: LT6654AMPS6-1.25, ul_LT6654AMPS6-1-25-TRMPBF:LT6654AMPS6-1.25-TRMPBF, F.Cu at (160.0, 169.5)
- added U33: ICL7660CSAT, ICL7660CSAT:SOIC127P600X175-8N, F.Cu at (146.5, 160.3)
- added U34: MSP430FR5969IRGZR, MSP430FR5969IRGZR:QFN50P700X700X100-49N, F.Cu at (62.5, 97.6)
- added U4: ADG841YKSZ-500RL7, ul_ADG841YKSZ-500RL7:ADG841YKSZ-500RL7, F.Cu at (200.5, 57.7)
- added U5: ADG841YKSZ-500RL7, ul_ADG841YKSZ-500RL7:ADG841YKSZ-500RL7, F.Cu at (200.5, 53.2)
- added U6: ADG841YKSZ-500RL7, ul_ADG841YKSZ-500RL7:ADG841YKSZ-500RL7, F.Cu at (200.5, 48.7)
- added U7: ADG841YKSZ-500RL7, ul_ADG841YKSZ-500RL7:ADG841YKSZ-500RL7, F.Cu at (200.5, 44.2)
- added U8: ADG841YKSZ-500RL7, ul_ADG841YKSZ-500RL7:ADG841YKSZ-500RL7, F.Cu at (200.5, 39.7)
- added U9: ADG841YKSZ-500RL7, ul_ADG841YKSZ-500RL7:ADG841YKSZ-500RL7, F.Cu at (200.5, 35.2)
- added Y1: CM8V-T1A, CM8V-T1A-32:XTAL_CM8V-T1A-32.768KHZ-7PF-20PPM-TA-QC, F.Cu at (61.5, 91.5)
Other:
- copper layers 2 -> 4
- net class Default: clearance 0.2 -> 0.1524; trace_width 0.25 -> 0.1524; via_dia 0.8 -> 0.508; via_drill 0.4 -> 0.254
- rule trace_clearance: 0.2 -> 0.1524
- rule trace_min: 0.2 -> 0.1524
- rule via_min_drill: 0.3 -> 0.254
- rule via_min_size: 0.4 -> 0.508
