File: flight_computer/flight_computer.sch (KiCad schematic (older format))
At the start: 0 parts

Commit message: Continuing layout
Changed lines of the file:
@@
 $Descr A3 16535 11693
 encoding utf-8
-Sheet 1 9
+Sheet 1 6
 Title ""
 Date ""
@@
 $EndDescr
 $Sheet
-S 10950 6500 1700 1350
+S 9100 6100 1700 1350
 U 635FEB2F
 F0 "Resistor Ladder" 50
 F1 "resistor_ladder.sch" 50
-F2 "V_PANEL" I R 12650 7150 50
-F3 "~LADDER_EN" I L 10950 6850 50
-F4 "LADDER_CLOCK" I L 10950 7000 50
-F5 "~LADDER_RESET" I L 10950 7150 50
-F6 "LADDER_LATCH" I L 10950 7300 50
-F7 "SCL" I L 10950 7500 50
-F8 "SDA" I L 10950 7600 50
+F2 "V_PANEL" I R 10800 6750 50
+F3 "~LADDER_EN" I L 9100 6450 50
+F4 "LADDER_CLOCK" I L 9100 6600 50
+F5 "~LADDER_RESET" I L 9100 6750 50
+F6 "LADDER_LATCH" I L 9100 6900 50
+F7 "SCL" I L 9100 7100 50
+F8 "SDA" I L 9100 7200 50
 $EndSheet
 $Sheet
-S 10950 4900 1700 1400
+S 9100 4500 1700 1400
 U 63C503EE
 F0 "Curve Tracer" 50
 F1 "curve_tracer.sch" 50
-F2 "PANEL_VOLTAGE" I R 12650 5500 50
-F3 "LADDER_VOLTAGE" I R 12650 5750 50
-F4 "SCLK" I L 10950 5150 50
-F5 "MOSI" I L 10950 5300 50
-F6 "MISO" I L 10950 5450 50
-F7 "ADC_CS" I L 10950 5600 50
-F8 "ADC_CLK" I L 10950 5750 50
-F9 "ADC_DRDY" I L 10950 5900 50
-F10 "ADC_SYNC" I L 10950 6050 50
+F2 "PANEL_VOLTAGE" I R 10800 5100 50
+F3 "LADDER_VOLTAGE" I R 10800 5350 50
+F4 "SCLK" I L 9100 4750 50
+F5 "MOSI" I L 9100 4900 50
+F6 "MISO" I L 9100 5050 50
+F7 "ADC_CS" I L 9100 5200 50
+F8 "ADC_CLK" I L 9100 5350 50
+F9 "ADC_DRDY" I L 9100 5500 50
+F10 "ADC_SYNC" I L 9100 5650 50
 $EndSheet
 $Sheet
-S 10950 2950 1700 1750
+S 9100 2550 1700 1750
 U 635FE71D
 F0 "Perovskite Switches" 50
 F1 "switcher.sch" 50
-F2 "ENABLE_TEST_SOURCE" I L 10950 4100 50
-F3 "RESET_PANEL_SWITCH" I L 10950 3250 50
-F4 "ENABLE_PANEL_SWITCH" I L 10950 3400 50
-F5 "10-19_CLOCK" I L 10950 3550 50
-F6 "0-9_CLOCK" I L 10950 3700 50
-F7 "PANEL_POSITIVE" O R 12650 3650 50
-F8 "REVERSE_BIAS" I L 10950 3950 50
-F9 "SDA" I L 10950 4400 50
-F10 "SCL" I L 10950 4300 50
+F2 "ENABLE_TEST_SOURCE" I L 9100 3700 50
+F3 "RESET_PANEL_SWITCH" I L 9100 2850 50
+F4 "ENABLE_PANEL_SWITCH" I L 9100 3000 50
+F5 "10-19_CLOCK" I L 9100 3150 50
+F6 "0-9_CLOCK" I L 9100 3300 50
+F7 "PANEL_POSITIVE" O R 10800 3250 50
+F8 "REVERSE_BIAS" I L 9100 3550 50
+F9 "SDA" I L 9100 4000 50
+F10 "SCL" I L 9100 3900 50
 $EndSheet
 $Sheet
-S 4650 2950 1700 650
-U 63D1F518
-F0 "Rad Hard Fault Watchdog" 50
-F1 "fault_watchdog.sch" 50
-F2 "FAULT" I R 6350 3400 50
-F3 "~PAYLOAD_RST" I R 6350 3200 50
-$EndSheet
-$Sheet
-S 7800 2950 1700 5900
+S 5950 2550 1700 5950
 U 63D21EEE
 F0 "Payload Controller" 50
 F1 "mission_payload.sch" 50
-F2 "~PAYLOAD_RST" I L 7800 3200 50
-F3 "FAULT" I L 7800 3400 50
-F4 "RESET_PANEL_SWITCH" I R 9500 3250 50
-F5 "ENABLE_PANEL_SWITCH" I R 9500 3400 50
-F6 "10-19_CLOCK" I R 9500 3550 50
-F7 "0-9_CLOCK" I R 9500 3700 50
-F8 "ENABLE_TEST_SOURCE" I R 9500 4100 50
-F9 "SCL" I R 9500 7500 50
-F10 "SDA" I R 9500 7600 50
-F11 "~LADDER_EN" I R 9500 6850 50
-F12 "LADDER_CLOCK" I R 9500 7000 50
-F13 "~LADDER_RESET" I R 9500 7150 50
-F14 "LADDER_LATCH" I R 9500 7300 50
-F15 "SCLK" I R 9500 5150 50
-F16 "MOSI" I R 9500 5300 50
-F17 "MISO" I R 9500 5450 50
-F18 "ADC_CLK" I R 9500 5750 50
-F19 "ADC_CS" I R 9500 5600 50
-F20 "ADC_DRDY" I R 9500 5900 50
-F21 "ADC_SYNC" I R 9500 6050 50
-F22 "RX_IN" O R 9500 8350 50
-F23 "TX_OUT" I R 9500 8500 50
-F24 "BUSY_IN" O R 9500 8650 50
-F25 "REVERSE_BIAS" I R 9500 3950 50
+F2 "RESET_PANEL_SWITCH" I R 7650 2850 50
+F3 "ENABLE_PANEL_SWITCH" I R 7650 3000 50
+F4 "10-19_CLOCK" I R 7650 3150 50
+F5 "0-9_CLOCK" I R 7650 3300 50
+F6 "ENABLE_TEST_SOURCE" I R 7650 3700 50
+F7 "SCL" I R 7650 7100 50
+F8 "SDA" I R 7650 7200 50
+F9 "~LADDER_EN" I R 7650 6450 50
+F10 "LADDER_CLOCK" I R 7650 6600 50
+F11 "~LADDER_RESET" I R 7650 6750 50
+F12 "LADDER_LATCH" I R 7650 6900 50
+F13 "SCLK" I R 7650 4750 50
+F14 "MOSI" I R 7650 4900 50
+F15 "MISO" I R 7650 5050 50
+F16 "ADC_CLK" I R 7650 5350 50
+F17 "ADC_CS" I R 7650 5200 50
+F18 "ADC_DRDY" I R 7650 5500 50
+F19 "ADC_SYNC" I R 7650 5650 50
+F20 "REVERSE_BIAS" I R 7650 3550 50
 $EndSheet
 $Sheet
-S 4650 4000 1700 1150
-U 63D2A1A8
-F0 "CubeSat Connections" 50
-F1 "cubesat.sch" 50
-$EndSheet
-$Sheet
-S 10950 1800 1700 850
+S 9100 7650 1700 850
 U 63D2A1C8
 F0 "Sun Sensor" 50
 F1 "sun_sensor.sch" 50
-F2 "SCL" I L 10950 2100 50
-F3 "SDA" I L 10950 2300 50
-$EndSheet
-$Sheet
-S 10950 8150 1700 700
-U 63D2A1FC
-F0 "Satellite Radio" 50
-F1 "sat_comms.sch" 50
-F2 "RX_IN" O L 10950 8350 50
-F3 "TX_OUT" I L 10950 8500 50
-F4 "BUSY_IN" O L 10950 8650 50
+F2 "SCL" I L 9100 8250 50
+F3 "SDA" I L 9100 7950 50
 $EndSheet
 Wire Wire Line
-	9500 7500 9900 7500
+	7650 7100 8050 7100
+Connection ~ 8050 7100
 Wire Wire Line
-	10950 7600 10050 7600
+	8050 7100 9100 7100
 Wire Wire Line
-	10950 2100 9900 2100
+	9100 3900 8050 3900
 Wire Wire Line
-	9900 2100 9900 4300
-Connection ~ 9900 7500
+	8050 3900 8050 7100
 Wire Wire Line
-	9900 7500 10950 7500
+	8150 4000 8150 7200
 Wire Wire Line
-	10950 2300 10050 2300
+	7650 2850 9100 2850
 Wire Wire Line
-	10050 2300 10050 4400
-Connection ~ 10050 7600
+	7650 3000 9100 3000
 Wire Wire Line
-	10050 7600 9500 7600
+	7650 3150 9100 3150
 Wire Wire Line
-	10950 4300 9900 4300
-Connection ~ 9900 4300
+	7650 3300 9100 3300
 Wire Wire Line
-	9900 4300 9900 7500
+	7650 3550 9100 3550
 Wire Wire Line
-	10950 4400 10050 4400
-Connection ~ 10050 4400
+	7650 3700 9100 3700
 Wire Wire Line
-	10050 4400 10050 7600
+	7650 4750 9100 4750
 Wire Wire Line
-	9500 3250 10950 3250
+	7650 4900 9100 4900
 Wire Wire Line
-	9500 3400 10950 3400
+	7650 5050 9100 5050
 Wire Wire Line
-	9500 3550 10950 3550
+	7650 5200 9100 5200
 Wire Wire Line
-	9500 3700 10950 3700
+	7650 5350 9100 5350
 Wire Wire Line
-	9500 3950 10950 3950
+	7650 5500 9100 5500
 Wire Wire Line
-	9500 4100 10950 4100
+	7650 5650 9100 5650
 Wire Wire Line
-	9500 5150 10950 5150
+	7650 6450 9100 6450
 Wire Wire Line
-	9500 5300 10950 5300
+	7650 6600 9100 6600
 Wire Wire Line
-	9500 5450 10950 5450
+	7650 6750 9100 6750
 Wire Wire Line
-	9500 5600 10950 5600
+	7650 6900 9100 6900
 Wire Wire Line
-	9500 5750 10950 5750
+	10800 3250 10900 3250
 Wire Wire Line
-	9500 5900 10950 5900
+	10900 3250 10900 5100
 Wire Wire Line
-	9500 6050 10950 6050
+	10900 5100 10800 5100
 Wire Wire Line
-	9500 6850 10950 6850
+	10800 5350 10900 5350
 Wire Wire Line
-	9500 7000 10950 7000
+	10900 5350 10900 6750
 Wire Wire Line
-	9500 7150 10950 7150
+	10900 6750 10800 6750
 Wire Wire Line
-	9500 7300 10950 7300
+	8150 7950 8150 7200
 Wire Wire Line
-	9500 8350 10950 8350
+	9100 8250 8050 8250
 Wire Wire Line
-	9500 8500 10950 8500
+	8050 8250 8050 7100
+Connection ~ 8150 7200
 Wire Wire Line
-	9500 8650 10950 8650
+	8150 7200 7650 7200
 Wire Wire Line
-	6350 3200 7800 3200
+	8150 7200 9100 7200
 Wire Wire Line
-	6350 3400 7800 3400
+	8150 7950 9100 7950
 Wire Wire Line
-	12650 3650 12750 3650
-Wire Wire Line
-	12750 3650 12750 5500
-Wire Wire Line
-	12750 5500 12650 5500
-Wire Wire Line
-	12650 5750 12750 5750
-Wire Wire Line
-	12750 5750 12750 7150
-Wire Wire Line
-	12750 7150 12650 7150
+	8150 4000 9100 4000
 $EndSCHEMATC
