File: flight_computer/switcher.sch (KiCad schematic (older format))
At the start: 59 parts, among them J3 G125-MV12605M1P, Q1 DMC2053UVT, U1 SN74LVC1G14DRL, U10 MAX4736EUBT, U11 MAX4736EUBT, U12 MAX4736EUBT, U13 MAX4736EUBT, U14 MAX4736EUBT, U15 LT3092ETS8TRPBF, U2 CD4518BM96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

Commit message: Working on flight computer
- Update resistor ladder curve tracer silkscreen, schematic, and layout
- Flight computer schematic drafted for MSP430 circuits, updated curve tracer, perovskite switching network.
Parts:
- removed J?: Panel Output to Curve Tracer, Connector_PinHeader_2.54mm:PinHeader_1x01_P2.54mm_Vertical, symbol Connector:Conn_01x01_Female
- added U?: MAX4736EUBT, MAX4736EUBT:SOP50P490X110-10N, symbol MAX4736EUBT:MAX4736EUBT
Connections:
- net labels added: PANEL_POSITIVE, REVERSE_BIAS, SCL, SDA
- wire segments 348 -> 317
Other:
- moved on the sheet: C?, J?, Q?A, Q?B, R?, U?

Commit message: Annotating schematic with references and footprints
Parts:
- removed U15: LT3092ETS8TRPBF, LT3092ETS8TRPBF:TSOT-23_TS8, symbol LT3092ETS8TRPBF:LT3092ETS8TRPBF
- added U30: LT3092EDD#TRPBF, LT3092EDD_TRPBF:DFN-8_DD, symbol LT3092EDD_TRPBF:LT3092EDD#TRPBF
- gave numbers to parts that had none: 2
Connections:
- wire segments 317 -> 318

Commit message: Continuing layout
Parts:
- added C46: 0.1u, Capacitor_SMD:C_0603_1608Metric, symbol Device:C
Connections:
- wire segments 318 -> 317
Changed lines of the file:
@@
 $Descr A2 23386 16535
 encoding utf-8
-Sheet 4 9
+Sheet 4 6
 Title "Perovskite Switching Circuit"
 Date "2022-09-24"
-Rev "A"
+Rev "B"
 Comp "Aerospace eXperimental Payloads | UNL Aerospace Club"
 Comment1 "Copyright (c) 2022"
@@
 Wire Wire Line
 	13000 11700 13000 2250
-Wire Wire Line
-	13000 2250 10650 2250
 $Comp
 L LT3092EDD_TRPBF:LT3092EDD#TRPBF U30
@@
 Wire Wire Line
 	12000 12950 12000 13050
+$Comp
+L Device:C C?
+U 1 1 638EC9CB
+P 5400 15150
+AR Path="/6313FC31/638EC9CB" Ref="C?"  Part="1"
+AR Path="/638EC9CB" Ref="C?"  Part="1"
+AR Path="/635FE71D/638EC9CB" Ref="C46"  Part="1"
+F 0 "C46" V 5652 15150 50  0000 C CNN
+F 1 "0.1u" V 5561 15150 50  0000 C CNN
+F 2 "Capacitor_SMD:C_0603_1608Metric" H 5438 15000 50  0001 C CNN
+F 3 "~" H 5400 15150 50  0001 C CNN
+	1    5400 15150
+	1    0    0    -1
+$EndComp
+$Comp
+L power:+3V3 #PWR?
+U 1 1 638EC9D1
+P 5400 15000
+AR Path="/6313FC31/638EC9D1" Ref="#PWR?"  Part="1"
+AR Path="/638EC9D1" Ref="#PWR?"  Part="1"
+AR Path="/635FE71D/638EC9D1" Ref="#PWR0152"  Part="1"
+F 0 "#PWR0152" H 5400 14850 50  0001 C CNN
+F 1 "+3V3" H 5415 15173 50  0000 C CNN
+F 2 "" H 5400 15000 50  0001 C CNN
+F 3 "" H 5400 15000 50  0001 C CNN
+	1    5400 15000
+	1    0    0    -1
+$EndComp
+$Comp
+L power:GND #PWR?
+U 1 1 638EC9D7
+P 5400 15300
+AR Path="/6313FC31/638EC9D7" Ref="#PWR?"  Part="1"
+AR Path="/638EC9D7" Ref="#PWR?"  Part="1"
+AR Path="/635FE71D/638EC9D7" Ref="#PWR0254"  Part="1"
+F 0 "#PWR0254" H 5400 15050 50  0001 C CNN
+F 1 "GND" H 5405 15127 50  0000 C CNN
+F 2 "" H 5400 15300 50  0001 C CNN
+F 3 "" H 5400 15300 50  0001 C CNN
+	1    5400 15300
+	1    0    0    -1
+$EndComp
 $EndSCHEMATC
