File: payload_controller/v2/switcher.sch (KiCad schematic (older format))
At the start: 62 parts, among them J1 GaAs Cell, J2 G125-MH12605M4R, J7 GaAs Temp, Q1 DMC2053UVT, U1 SN74LVC1G14DRL, U10 MAX4736EUBT, U11 MAX4736EUBT, U12 MAX4736EUBT, U13 MAX4736EUBT, U14 74LVC1G332, U14 MAX4736EUBT, U19 MAX4736EUBT, U2 CD4518BM96, U3 CD4028BMT, U30 LT3092EDD#TRPBF, U4 CD4028BMT, U5 MAX4736EUBT, U6 MAX4736EUBT, U7 MAX4736EUBT, U8 MAX4736EUBT, U9 MAX4736EUBT

Commit message: Finish updated switcher
Connections:
- net GND: no longer R10.1, R11.1, R12.1, R13.1, R14.1, R15.1, R16.1, R17.1, R18.1, R19.1, R20.1, R21.1, R4.1, R5.1, R6.1, R7.1, R8.1, R9.1
- net PANEL_POSITIVE: now also R10.1, R11.1, R12.1, R13.1, R14.1, R15.1, R16.1, R17.1, R18.1, R19.1, R20.1, R21.1, R4.1, R5.1, R6.1, R7.1, R8.1, R9.1
Changed lines of the file:
@@
 Wire Wire Line
 	10650 11700 10850 11700
-Connection ~ 11600 11600
-Wire Wire Line
-	11600 11600 11600 11800
 Wire Wire Line
 	11600 11300 11600 11600
@@
 	11500 11300 11600 11300
 Wire Wire Line
-	11600 10650 11600 10850
-Connection ~ 11600 10650
-Wire Wire Line
 	11500 10650 11600 10650
 Wire Wire Line
@@
 	11500 10350 11600 10350
 Wire Wire Line
-	11600 9700 11600 9900
-Connection ~ 11600 9700
-Wire Wire Line
 	11500 9700 11600 9700
 Wire Wire Line
@@
 	11500 9400 11600 9400
 Wire Wire Line
-	11600 8750 11600 8950
-Connection ~ 11600 8750
-Wire Wire Line
 	11500 8750 11600 8750
 Wire Wire Line
@@
 	11500 8450 11600 8450
 Wire Wire Line
-	11600 7800 11600 8000
-Connection ~ 11600 7800
-Wire Wire Line
 	11500 7800 11600 7800
 Wire Wire Line
@@
 	11500 7500 11600 7500
 Wire Wire Line
-	11600 6850 11600 7050
-Connection ~ 11600 6850
-Wire Wire Line
 	11500 6850 11600 6850
 Wire Wire Line
@@
 	11500 6550 11600 6550
 Wire Wire Line
-	11600 5900 11600 6100
-Connection ~ 11600 5900
-Wire Wire Line
 	11500 5900 11600 5900
 Wire Wire Line
@@
 	11500 5600 11600 5600
 Wire Wire Line
-	11600 4950 11600 5150
-Connection ~ 11600 4950
-Wire Wire Line
 	11500 4950 11600 4950
 Wire Wire Line
@@
 	11500 4650 11600 4650
 Wire Wire Line
-	11600 4000 11600 4200
-Connection ~ 11600 4000
-Wire Wire Line
 	11500 4000 11600 4000
 Wire Wire Line
@@
 	11500 3700 11600 3700
 Wire Wire Line
-	11600 3050 11600 3250
-Connection ~ 11600 3050
-Wire Wire Line
 	11500 3050 11600 3050
 Wire Wire Line
@@
 Wire Wire Line
 	11500 2750 11600 2750
-$Comp
-L power:GND #PWR?
-U 1 1 6387CB57
-P 11600 11800
-AR Path="/6313FC31/6387CB57" Ref="#PWR?"  Part="1"
-AR Path="/6387CB57" Ref="#PWR0140"  Part="1"
-AR Path="/635FE71D/6387CB57" Ref="#PWR0205"  Part="1"
-F 0 "#PWR0205" H 11600 11550 50  0001 C CNN
-F 1 "GND" H 11605 11627 50  0000 C CNN
-F 2 "" H 11600 11800 50  0001 C CNN
-F 3 "" H 11600 11800 50  0001 C CNN
-	1    11600 11800
-	1    0    0    -1
-$EndComp
-$Comp
-L power:GND #PWR?
-U 1 1 6387CB51
-P 11600 10850
-AR Path="/6313FC31/6387CB51" Ref="#PWR?"  Part="1"
-AR Path="/6387CB51" Ref="#PWR0139"  Part="1"
-AR Path="/635FE71D/6387CB51" Ref="#PWR0204"  Part="1"
-F 0 "#PWR0204" H 11600 10600 50  0001 C CNN
-F 1 "GND" H 11605 10677 50  0000 C CNN
-F 2 "" H 11600 10850 50  0001 C CNN
-F 3 "" H 11600 10850 50  0001 C CNN
-	1    11600 10850
-	1    0    0    -1
-$EndComp
-$Comp
-L power:GND #PWR?
-U 1 1 6387CB4B
-P 11600 9900
-AR Path="/6313FC31/6387CB4B" Ref="#PWR?"  Part="1"
-AR Path="/6387CB4B" Ref="#PWR0138"  Part="1"
-AR Path="/635FE71D/6387CB4B" Ref="#PWR0203"  Part="1"
-F 0 "#PWR0203" H 11600 9650 50  0001 C CNN
-F 1 "GND" H 11605 9727 50  0000 C CNN
-F 2 "" H 11600 9900 50  0001 C CNN
-F 3 "" H 11600 9900 50  0001 C CNN
-	1    11600 9900
-	1    0    0    -1
-$EndComp
-$Comp
-L power:GND #PWR?
-U 1 1 6387CB45
-P 11600 8950
-AR Path="/6313FC31/6387CB45" Ref="#PWR?"  Part="1"
-AR Path="/6387CB45" Ref="#PWR0137"  Part="1"
-AR Path="/635FE71D/6387CB45" Ref="#PWR0202"  Part="1"
-F 0 "#PWR0202" H 11600 8700 50  0001 C CNN
-F 1 "GND" H 11605 8777 50  0000 C CNN
-F 2 "" H 11600 8950 50  0001 C CNN
-F 3 "" H 11600 8950 50  0001 C CNN
-	1    11600 8950
-	1    0    0    -1
-$EndComp
-$Comp
-L power:GND #PWR?
-U 1 1 6387CB3F
-P 11600 8000
-AR Path="/6313FC31/6387CB3F" Ref="#PWR?"  Part="1"
-AR Path="/6387CB3F" Ref="#PWR0136"  Part="1"
-AR Path="/635FE71D/6387CB3F" Ref="#PWR0201"  Part="1"
-F 0 "#PWR0201" H 11600 7750 50  0001 C CNN
-F 1 "GND" H 11605 7827 50  0000 C CNN
-F 2 "" H 11600 8000 50  0001 C CNN
-F 3 "" H 11600 8000 50  0001 C CNN
-	1    11600 8000
-	1    0    0    -1
-$EndComp
-$Comp
-L power:GND #PWR?
-U 1 1 6387CB39
-P 11600 7050
-AR Path="/6313FC31/6387CB39" Ref="#PWR?"  Part="1"
-AR Path="/6387CB39" Ref="#PWR0135"  Part="1"
-AR Path="/635FE71D/6387CB39" Ref="#PWR0200"  Part="1"
-F 0 "#PWR0200" H 11600 6800 50  0001 C CNN
-F 1 "GND" H 11605 6877 50  0000 C CNN
-F 2 "" H 11600 7050 50  0001 C CNN
-F 3 "" H 11600 7050 50  0001 C CNN
-	1    11600 7050
-	1    0    0    -1
-$EndComp
-$Comp
-L power:GND #PWR?
-U 1 1 6387CB33
-P 11600 6100
-AR Path="/6313FC31/6387CB33" Ref="#PWR?"  Part="1"
-AR Path="/6387CB33" Ref="#PWR0134"  Part="1"
-AR Path="/635FE71D/6387CB33" Ref="#PWR0199"  Part="1"
-F 0 "#PWR0199" H 11600 5850 50  0001 C CNN
-F 1 "GND" H 11605 5927 50  0000 C CNN
-F 2 "" H 11600 6100 50  0001 C CNN
-F 3 "" H 11600 6100 50  0001 C CNN
-	1    11600 6100
-	1    0    0    -1
-$EndComp
-$Comp
-L power:GND #PWR?
-U 1 1 6387CB2D
-P 11600 5150
-AR Path="/6313FC31/6387CB2D" Ref="#PWR?"  Part="1"
-AR Path="/6387CB2D" Ref="#PWR0133"  Part="1"
-AR Path="/635FE71D/6387CB2D" Ref="#PWR0198"  Part="1"
-F 0 "#PWR0198" H 11600 4900 50  0001 C CNN
-F 1 "GND" H 11605 4977 50  0000 C CNN
-F 2 "" H 11600 5150 50  0001 C CNN
-F 3 "" H 11600 5150 50  0001 C CNN
-	1    11600 5150
-	1    0    0    -1
-$EndComp
-$Comp
-L power:GND #PWR?
-U 1 1 6387CB27
-P 11600 3250
-AR Path="/6313FC31/6387CB27" Ref="#PWR?"  Part="1"
-AR Path="/6387CB27" Ref="#PWR0132"  Part="1"
-AR Path="/635FE71D/6387CB27" Ref="#PWR0197"  Part="1"
-F 0 "#PWR0197" H 11600 3000 50  0001 C CNN
-F 1 "GND" H 11605 3077 50  0000 C CNN
-F 2 "" H 11600 3250 50  0001 C CNN
-F 3 "" H 11600 3250 50  0001 C CNN
-	1    11600 3250
-	1    0    0    -1
-$EndComp
-$Comp
-L power:GND #PWR?
-U 1 1 6387CB21
-P 11600 4200
-AR Path="/6313FC31/6387CB21" Ref="#PWR?"  Part="1"
-AR Path="/6387CB21" Ref="#PWR0131"  Part="1"
-AR Path="/635FE71D/6387CB21" Ref="#PWR0196"  Part="1"
-F 0 "#PWR0196" H 11600 3950 50  0001 C CNN
-F 1 "GND" H 11605 4027 50  0000 C CNN
-F 2 "" H 11600 4200 50  0001 C CNN
-F 3 "" H 11600 4200 50  0001 C CNN
-	1    11600 4200
-	1    0    0    -1
-$EndComp
 Wire Wire Line
 	10650 11600 11200 11600
@@
 	13250 11000 13150 11000
 Wire Wire Line
-	11000 1850 12200 1850
+	11000 1850 11600 1850
 Wire Wire Line
 	15650 10900 15650 11050
@@
 	1    0    0    -1
 $EndComp
+$Comp
+L power:GND #PWR?
+U 1 1 6387CB57
+P 11600 11800
+AR Path="/6313FC31/6387CB57" Ref="#PWR?"  Part="1"
+AR Path="/6387CB57" Ref="#PWR0140"  Part="1"
+AR Path="/635FE71D/6387CB57" Ref="#PWR0205"  Part="1"
+F 0 "#PWR0205" H 11600 11550 50  0001 C CNN
+F 1 "GND" H 11605 11627 50  0000 C CNN
+F 2 "" H 11600 11800 50  0001 C CNN
+F 3 "" H 11600 11800 50  0001 C CNN
+	1    11600 11800
+	1    0    0    -1
+$EndComp
+Connection ~ 11600 11600
+Wire Wire Line
+	11600 11600 11600 11800
+Wire Wire Line
+	11600 1850 11600 2750
+Connection ~ 11600 1850
+Wire Wire Line
+	11600 1850 12200 1850
+Connection ~ 11600 2750
+Wire Wire Line
+	11600 3050 11600 3700
+Connection ~ 11600 3050
+Connection ~ 11600 3700
+Wire Wire Line
+	11600 4000 11600 4650
+Connection ~ 11600 4000
+Connection ~ 11600 4650
+Wire Wire Line
+	11600 4950 11600 5600
+Connection ~ 11600 4950
+Connection ~ 11600 5600
+Wire Wire Line
+	11600 5900 11600 6550
+Connection ~ 11600 5900
+Connection ~ 11600 6550
+Wire Wire Line
+	11600 6850 11600 7500
+Connection ~ 11600 6850
+Connection ~ 11600 7500
+Wire Wire Line
+	11600 7800 11600 8450
+Connection ~ 11600 7800
+Connection ~ 11600 8450
+Wire Wire Line
+	11600 8750 11600 9400
+Connection ~ 11600 8750
+Connection ~ 11600 9400
+Wire Wire Line
+	11600 9700 11600 10350
+Connection ~ 11600 9700
+Connection ~ 11600 10350
 $EndSCHEMATC
