File: NREL_tester/multiplexer cell tester/multiplexer cell tester.sch (KiCad schematic (older format))
At the start: 11 parts

Commit message: Review contact board
Parts:
- U1: renamed from U?; footprint Package_TO_SOT_SMD:SOT-553 -> Package_TO_SOT_SMD:SOT-23-5
- gave numbers to parts that had none: 10
Connections:
- net 10-19_CLOCK: now also R4.2; no longer R6.1
- net ENABLE_PANEL_SWITCH: now also R5.1; no longer R7.1
- net GND: now also J2.1 (Pin_1); no longer J2.10 (Pin_10)
- net PANEL_2: now also J2.3 (Pin_3); no longer J2.8 (Pin_8)
- net PANEL_3: now also J2.2 (Pin_2); no longer J2.9 (Pin_9)
- net RESET_PANEL_SWITCH: now also R6.1; no longer R4.2
- net REVERSE_BIAS: now also R7.1; no longer R5.1
- net at R4.1: now also J2.9 (Pin_9); no longer J2.2 (Pin_2)
- net at R6.2: now also J2.7 (Pin_7); no longer J2.4 (Pin_4)
- net at R7.2: now also J2.6 (Pin_6); no longer J2.5 (Pin_5)
- net at R3.1: now also J2.10 (Pin_10); no longer J2.1 (Pin_1)
- net at R5.2: now also J2.8 (Pin_8); no longer J2.3 (Pin_3)
Changed lines of the file:
@@
 encoding utf-8
 Sheet 1 5
-Title ""
-Date ""
-Rev ""
-Comp ""
-Comment1 ""
-Comment2 ""
-Comment3 ""
-Comment4 ""
+Title "IV Curve Tracer for Ossila AM1.5 Solar Simulator"
+Date "2023-07-08"
+Rev "A"
+Comp "Aerospace eXperimental Payloads | UNL Aerospace Club"
+Comment1 "Copyright (c) 2023"
+Comment2 "Designer: WSA"
+Comment3 "Reviewer: WSA"
+Comment4 "Approved: WSA"
 $EndDescr
 $Sheet
@@
 P 2550 5100
 AR Path="/6313FC31/64966A3F" Ref="R?"  Part="1"
-AR Path="/64966A3F" Ref="R?"  Part="1"
+AR Path="/64966A3F" Ref="R4"  Part="1"
 AR Path="/648F7944/64966A3F" Ref="R?"  Part="1"
-F 0 "R?" V 2550 5550 50  0000 C CNN
+F 0 "R4" V 2550 5550 50  0000 C CNN
 F 1 "100" V 2550 5100 50  0000 C CNN
 F 2 "Resistor_SMD:R_0603_1608Metric" V 2480 5100 50  0001 C CNN
@@
 P 2550 5300
 AR Path="/6313FC31/64966A45" Ref="R?"  Part="1"
-AR Path="/64966A45" Ref="R?"  Part="1"
+AR Path="/64966A45" Ref="R6"  Part="1"
 AR Path="/648F7944/64966A45" Ref="R?"  Part="1"
-F 0 "R?" V 2550 4850 50  0000 C CNN
+F 0 "R6" V 2550 4850 50  0000 C CNN
 F 1 "100" V 2550 5300 50  0000 C CNN
 F 2 "Resistor_SMD:R_0603_1608Metric" V 2480 5300 50  0001 C CNN
@@
 P 2550 5400
 AR Path="/6313FC31/64966A4B" Ref="R?"  Part="1"
-AR Path="/64966A4B" Ref="R?"  Part="1"
+AR Path="/64966A4B" Ref="R7"  Part="1"
 AR Path="/648F7944/64966A4B" Ref="R?"  Part="1"
-F 0 "R?" V 2550 4950 50  0000 C CNN
+F 0 "R7" V 2550 4950 50  0000 C CNN
 F 1 "100" V 2550 5400 50  0000 C CNN
 F 2 "Resistor_SMD:R_0603_1608Metric" V 2480 5400 50  0001 C CNN
@@
 P 2550 3700
 AR Path="/648F7944/64966A51" Ref="FB?"  Part="1"
-AR Path="/64966A51" Ref="FB?"  Part="1"
-F 0 "FB?" H 2687 3746 50  0000 L CNN
+AR Path="/64966A51" Ref="FB1"  Part="1"
+F 0 "FB1" H 2687 3746 50  0000 L CNN
 F 1 "Ferrite_Bead" H 2687 3655 50  0000 L CNN
 F 2 "Inductor_SMD:L_0603_1608Metric" V 2480 3700 50  0001 C CNN
@@
 	1    0    0    -1
 $EndComp
-Text GLabel 2700 5300 2    50   Input ~ 0
+Text GLabel 2700 5100 2    50   Input ~ 0
 10-19_CLOCK
-Text GLabel 2700 5400 2    50   Input ~ 0
+Text GLabel 2700 5200 2    50   Input ~ 0
 ENABLE_PANEL_SWITCH
 Wire Wire Line
@@
 P 2550 3400
 AR Path="/6313FC31/64966A5F" Ref="#PWR?"  Part="1"
-AR Path="/64966A5F" Ref="#PWR?"  Part="1"
+AR Path="/64966A5F" Ref="#PWR0101"  Part="1"
 AR Path="/648F7944/64966A5F" Ref="#PWR?"  Part="1"
-F 0 "#PWR?" H 2550 3250 50  0001 C CNN
+F 0 "#PWR0101" H 2550 3250 50  0001 C CNN
 F 1 "+3V3" H 2565 3573 50  0000 C CNN
 F 2 "" H 2550 3400 50  0001 C CNN
@@
 P 2550 6050
 AR Path="/6313FC31/64966A65" Ref="#PWR?"  Part="1"
-AR Path="/64966A65" Ref="#PWR?"  Part="1"
+AR Path="/64966A65" Ref="#PWR0102"  Part="1"
 AR Path="/648F7944/64966A65" Ref="#PWR?"  Part="1"
-F 0 "#PWR?" H 2550 5800 50  0001 C CNN
+F 0 "#PWR0102" H 2550 5800 50  0001 C CNN
 F 1 "GND" H 2555 5877 50  0000 C CNN
 F 2 "" H 2550 6050 50  0001 C CNN
@@
 $Comp
 L Connector:Conn_01x10_Female J?
-U 1 1 64966A6B
-P 2200 5400
-AR Path="/648F7944/64966A6B" Ref="J?"  Part="1"
-AR Path="/64966A6B" Ref="J?"  Part="1"
-F 0 "J?" H 2100 5950 50  0000 C CNN
-F 1 "Conn_01x10_Female" H 2092 4766 50  0001 C CNN
-F 2 "Connector_PinHeader_2.54mm:PinHeader_1x10_P2.54mm_Vertical" H 2200 5400 50  0001 C CNN
-F 3 "~" H 2200 5400 50  0001 C CNN
-	1    2200 5400
-	-1   0    0    -1
-$EndComp
-$Comp
-L Connector:Conn_01x10_Female J?
 U 1 1 64966A71
 P 2200 4250
 AR Path="/648F7944/64966A71" Ref="J?"  Part="1"
-AR Path="/64966A71" Ref="J?"  Part="1"
-F 0 "J?" H 2092 4743 50  0000 C CNN
+AR Path="/64966A71" Ref="J1"  Part="1"
+F 0 "J1" H 2092 4743 50  0000 C CNN
 F 1 "Conn_01x10_Female" H 2092 3616 50  0001 C CNN
 F 2 "Connector_PinHeader_2.54mm:PinHeader_1x10_P2.54mm_Vertical" H 2200 4250 50  0001 C CNN
@@
 P 2550 5200
 AR Path="/6313FC31/64966A86" Ref="R?"  Part="1"
-AR Path="/64966A86" Ref="R?"  Part="1"
+AR Path="/64966A86" Ref="R5"  Part="1"
 AR Path="/648F7944/64966A86" Ref="R?"  Part="1"
-F 0 "R?" V 2550 4750 50  0000 C CNN
+F 0 "R5" V 2550 4750 50  0000 C CNN
 F 1 "100" V 2550 5200 50  0000 C CNN
 F 2 "Resistor_SMD:R_0603_1608Metric" V 2480 5200 50  0001 C CNN
@@
 	0    1    1    0
 $EndComp
-Text GLabel 2700 5200 2    50   Input ~ 0
+Text GLabel 2700 5400 2    50   Input ~ 0
 REVERSE_BIAS
 $Sheet
@@
 Text GLabel 4700 1900 0    50   Input ~ 0
 10-19_CLOCK
-Text GLabel 2700 5100 2    50   Input ~ 0
+Text GLabel 2700 5300 2    50   Input ~ 0
 RESET_PANEL_SWITCH
 Text GLabel 4700 2200 0    50   Input ~ 0
@@
 P 4650 2650
 AR Path="/6313FC31/64A640C4" Ref="#PWR?"  Part="1"
-AR Path="/64A640C4" Ref="#PWR?"  Part="1"
+AR Path="/64A640C4" Ref="#PWR0103"  Part="1"
 AR Path="/648F7944/64A640C4" Ref="#PWR?"  Part="1"
-F 0 "#PWR?" H 4650 2400 50  0001 C CNN
+F 0 "#PWR0103" H 4650 2400 50  0001 C CNN
 F 1 "GND" H 4655 2477 50  0000 C CNN
 F 2 "" H 4650 2650 50  0001 C CNN
@@
 P 8150 4200
 AR Path="/6313FC31/64B78CD3" Ref="#PWR?"  Part="1"
-AR Path="/64B78CD3" Ref="#PWR?"  Part="1"
+AR Path="/64B78CD3" Ref="#PWR0104"  Part="1"
 AR Path="/648F7944/64B78CD3" Ref="#PWR?"  Part="1"
-F 0 "#PWR?" H 8150 3950 50  0001 C CNN
+F 0 "#PWR0104" H 8150 3950 50  0001 C CNN
 F 1 "GND" H 8155 4027 50  0000 C CNN
 F 2 "" H 8150 4200 50  0001 C CNN
@@
 P 2550 5000
 AR Path="/6313FC31/64B7E372" Ref="R?"  Part="1"
-AR Path="/64B7E372" Ref="R?"  Part="1"
+AR Path="/64B7E372" Ref="R3"  Part="1"
 AR Path="/648F7944/64B7E372" Ref="R?"  Part="1"
-F 0 "R?" V 2550 5450 50  0000 C CNN
+F 0 "R3" V 2550 5450 50  0000 C CNN
 F 1 "100" V 2550 5000 50  0000 C CNN
 F 2 "Resistor_SMD:R_0603_1608Metric" V 2480 5000 50  0001 C CNN
@@
 P 2550 4450
 AR Path="/6313FC31/64B7F6B2" Ref="R?"  Part="1"
-AR Path="/64B7F6B2" Ref="R?"  Part="1"
+AR Path="/64B7F6B2" Ref="R1"  Part="1"
 AR Path="/648F7944/64B7F6B2" Ref="R?"  Part="1"
-F 0 "R?" V 2550 4900 50  0000 C CNN
+F 0 "R1" V 2550 4900 50  0000 C CNN
 F 1 "100" V 2550 4450 50  0000 C CNN
 F 2 "Resistor_SMD:R_0603_1608Metric" V 2480 4450 50  0001 C CNN
@@
 P 2550 4550
 AR Path="/6313FC31/64B8035D" Ref="R?"  Part="1"
-AR Path="/64B8035D" Ref="R?"  Part="1"
+AR Path="/64B8035D" Ref="R2"  Part="1"
 AR Path="/648F7944/64B8035D" Ref="R?"  Part="1"
-F 0 "R?" V 2550 5000 50  0000 C CNN
+F 0 "R2" V 2550 5000 50  0000 C CNN
 F 1 "100" V 2550 4550 50  0000 C CNN
 F 2 "Resistor_SMD:R_0603_1608Metric" V 2480 4550 50  0001 C CNN
@@
 U 1 1 64BA669B
 P 6400 3700
-F 0 "U?" H 6450 3600 50  0000 L CNN
+AR Path="/648F7944/64BA669B" Ref="U?"  Part="1"
+AR Path="/64BA669B" Ref="U1"  Part="1"
+F 0 "U1" H 6450 3600 50  0000 L CNN
 F 1 "SN74LVC1G14DRL" H 6450 3500 50  0000 L CNN
-F 2 "Package_TO_SOT_SMD:SOT-553" H 6400 3450 50  0001 C CNN
+F 2 "Package_TO_SOT_SMD:SOT-23-5" H 6400 3450 50  0001 C CNN
 F 3 "http://www.ti.com/lit/ds/symlink/sn74lvc1g14.pdf" H 6400 3700 50  0001 C CNN
 	1    6400 3700
@@
 P 6400 4050
 AR Path="/6313FC31/64BA6AF4" Ref="#PWR?"  Part="1"
-AR Path="/64BA6AF4" Ref="#PWR?"  Part="1"
+AR Path="/64BA6AF4" Ref="#PWR0105"  Part="1"
 AR Path="/648F7944/64BA6AF4" Ref="#PWR?"  Part="1"
-F 0 "#PWR?" H 6400 3800 50  0001 C CNN
+F 0 "#PWR0105" H 6400 3800 50  0001 C CNN
 F 1 "GND" H 6405 3877 50  0000 C CNN
 F 2 "" H 6400 4050 50  0001 C CNN
@@
 P 6400 3500
 AR Path="/6313FC31/64BA6EDC" Ref="#PWR?"  Part="1"
-AR Path="/64BA6EDC" Ref="#PWR?"  Part="1"
+AR Path="/64BA6EDC" Ref="#PWR0106"  Part="1"
 AR Path="/648F7944/64BA6EDC" Ref="#PWR?"  Part="1"
-F 0 "#PWR?" H 6400 3350 50  0001 C CNN
+F 0 "#PWR0106" H 6400 3350 50  0001 C CNN
 F 1 "+3V3" H 6415 3673 50  0000 C CNN
 F 2 "" H 6400 3500 50  0001 C CNN
@@
 Wire Wire Line
 	6150 4000 8300 4000
+$Comp
+L Connector:Conn_01x10_Female J?
+U 1 1 64966A6B
+P 2200 5500
+AR Path="/648F7944/64966A6B" Ref="J?"  Part="1"
+AR Path="/64966A6B" Ref="J2"  Part="1"
+F 0 "J2" H 2100 6050 50  0000 C CNN
+F 1 "Conn_01x10_Female" H 2092 4866 50  0001 C CNN
+F 2 "Connector_PinHeader_2.54mm:PinHeader_1x10_P2.54mm_Vertical" H 2200 5500 50  0001 C CNN
+F 3 "~" H 2200 5500 50  0001 C CNN
+	1    2200 5500
+	-1   0    0    1
+$EndComp
 $EndSCHEMATC
