File: flight_computer/v2/curve_tracer.sch (KiCad schematic (older format))
At the start: 73 parts, among them U1 OPA2387, U10 OPA2387, U10 TLV7031DBV, U11 INA190A4IDDFR, U12 INA190A4IDDFR, U13 INA190A4IDDFR, U14 INA190A4IDDFR, U2 OPA2387, U9 SN74CBT3253

Commit message: Finished layout of flight computer
Parts:
- removed C17, C18: 0.1u, Capacitor_SMD:C_0603_1608Metric, symbol Device:C
- removed TP11, TP19, TP21, TP3: Voltage Test-, TestPoint:TestPoint_Pad_1.0x1.0mm, symbol Connector:TestPoint
- added TP9: Voltage Test+, TestPoint:TestPoint_Pad_1.0x1.0mm, symbol Connector:TestPoint
Connections:
- net +3V3: now also C16.1, C16.1, C20.1, C21.1
- net P_1_CURRENT: now also U9.3 (1B4); no longer U9.5 (1B2)
- net P_1_VOLTAGE: now also U9.13 (2B4); no longer U9.11 (2B2)
- net P_3_CURRENT: now also U9.5 (1B2); no longer U9.3 (1B4)
- net P_3_VOLTAGE: now also U9.11 (2B2); no longer U9.13 (2B4)
- net VBUS: no longer C16.1, C16.1, C20.1, C21.1
- net at R4.2, R5.1, U10.4 (-): now also TP9.1
