File: flight_computer/v2/eps_connections.sch (KiCad schematic (older format))
At the start: 30 parts, among them J15 Power, J16 Power, J17 Power, J18 Power, J19 Power, J20 BUSS+, J21 EPS Serial, J22 Power, Q1 BSS138, Q2 BSS138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

Commit message: Finished layout of flight computer
Parts:
- removed C102: 10u, Capacitor_SMD:C_0603_1608Metric, symbol Device:C
- removed C103: 0.1u, Capacitor_SMD:C_0603_1608Metric, symbol Device:C
- removed J17: Power, Connector_Hirose:Hirose_DF13C_CL535-0402-2-51_1x02-1MP_P1.25mm_Vertical, symbol Connector:Conn_01x02_Male
Connections:
- net VDDF: no longer C101.1
- net VPP: now also C101.1
Changed lines of the file:
@@
 $Descr A4 11693 8268
 encoding utf-8
-Sheet 7 8
+Sheet 6 8
 Title "EPS Connections"
 Date "2023-08-13"
@@
 $Comp
 L Connector:Conn_01x02_Male J?
-U 1 1 6686117D
-P 5700 4550
-AR Path="/64D823E8/6686117D" Ref="J?"  Part="1"
-AR Path="/64D821F3/6686117D" Ref="J17"  Part="1"
-F 0 "J17" H 5672 4524 50  0000 R CNN
-F 1 "Power" H 5672 4433 50  0000 R CNN
-F 2 "Connector_Hirose:Hirose_DF13C_CL535-0402-2-51_1x02-1MP_P1.25mm_Vertical" H 5700 4550 50  0001 C CNN
-F 3 "~" H 5700 4550 50  0001 C CNN
-	1    5700 4550
-	-1   0    0    -1
-$EndComp
-$Comp
-L power:GND #PWR?
-U 1 1 66861183
-P 5500 4650
-AR Path="/6313FC31/66861183" Ref="#PWR?"  Part="1"
-AR Path="/66861183" Ref="#PWR?"  Part="1"
-AR Path="/648F7944/66861183" Ref="#PWR?"  Part="1"
-AR Path="/64A6B33A/66861183" Ref="#PWR?"  Part="1"
-AR Path="/64D823E8/66861183" Ref="#PWR?"  Part="1"
-AR Path="/64D821F3/66861183" Ref="#PWR0335"  Part="1"
-F 0 "#PWR0335" H 5500 4400 50  0001 C CNN
-F 1 "GND" H 5505 4477 50  0000 C CNN
-F 2 "" H 5500 4650 50  0001 C CNN
-F 3 "" H 5500 4650 50  0001 C CNN
-	1    5500 4650
-	1    0    0    -1
-$EndComp
-$Comp
-L Connector:Conn_01x02_Male J?
 U 1 1 66862097
 P 5050 4550
@@
 $EndComp
 $Comp
-L power:VDDA #PWR0334
-U 1 1 6686295A
-P 5500 4550
-F 0 "#PWR0334" H 5500 4400 50  0001 C CNN
-F 1 "VDDA" H 5515 4723 50  0000 C CNN
-F 2 "" H 5500 4550 50  0001 C CNN
-F 3 "" H 5500 4550 50  0001 C CNN
-	1    5500 4550
-	1    0    0    -1
-$EndComp
-$Comp
 L power:VDDF #PWR0326
 U 1 1 6686361F
@@
 F 3 "" H 4850 4550 50  0001 C CNN
 	1    4850 4550
-	1    0    0    -1
-$EndComp
-$Comp
-L Device:C C103
-U 1 1 668B1987
-P 5050 5500
-F 0 "C103" H 5165 5546 50  0000 L CNN
-F 1 "0.1u" H 5165 5455 50  0000 L CNN
-F 2 "Capacitor_SMD:C_0603_1608Metric" H 5088 5350 50  0001 C CNN
-F 3 "~" H 5050 5500 50  0001 C CNN
-	1    5050 5500
-	1    0    0    -1
-$EndComp
-$Comp
-L power:GND #PWR?
-U 1 1 668B198D
-P 5050 5650
-AR Path="/6313FC31/668B198D" Ref="#PWR?"  Part="1"
-AR Path="/668B198D" Ref="#PWR?"  Part="1"
-AR Path="/648F7944/668B198D" Ref="#PWR?"  Part="1"
-AR Path="/64A6B33A/668B198D" Ref="#PWR?"  Part="1"
-AR Path="/64D823E8/668B198D" Ref="#PWR?"  Part="1"
-AR Path="/64D821F3/668B198D" Ref="#PWR0330"  Part="1"
-F 0 "#PWR0330" H 5050 5400 50  0001 C CNN
-F 1 "GND" H 5055 5477 50  0000 C CNN
-F 2 "" H 5050 5650 50  0001 C CNN
-F 3 "" H 5050 5650 50  0001 C CNN
-	1    5050 5650
-	1    0    0    -1
-$EndComp
-$Comp
-L Device:C C102
-U 1 1 668B1999
-P 4650 5500
-F 0 "C102" H 4765 5546 50  0000 L CNN
-F 1 "10u" H 4765 5455 50  0000 L CNN
-F 2 "Capacitor_SMD:C_0603_1608Metric" H 4688 5350 50  0001 C CNN
-F 3 "~" H 4650 5500 50  0001 C CNN
-	1    4650 5500
-	1    0    0    -1
-$EndComp
-$Comp
-L power:GND #PWR?
-U 1 1 668B199F
-P 4650 5650
-AR Path="/6313FC31/668B199F" Ref="#PWR?"  Part="1"
-AR Path="/668B199F" Ref="#PWR?"  Part="1"
-AR Path="/648F7944/668B199F" Ref="#PWR?"  Part="1"
-AR Path="/64A6B33A/668B199F" Ref="#PWR?"  Part="1"
-AR Path="/64D823E8/668B199F" Ref="#PWR?"  Part="1"
-AR Path="/64D821F3/668B199F" Ref="#PWR0325"  Part="1"
-F 0 "#PWR0325" H 4650 5400 50  0001 C CNN
-F 1 "GND" H 4655 5477 50  0000 C CNN
-F 2 "" H 4650 5650 50  0001 C CNN
-F 3 "" H 4650 5650 50  0001 C CNN
-	1    4650 5650
 	1    0    0    -1
 $EndComp
@@
 F 3 "" H 3850 5350 50  0001 C CNN
 	1    3850 5350
-	1    0    0    -1
-$EndComp
-$Comp
-L power:VDDF #PWR0321
-U 1 1 668B41AA
-P 4250 5350
-F 0 "#PWR0321" H 4250 5200 50  0001 C CNN
-F 1 "VDDF" H 4265 5523 50  0000 C CNN
-F 2 "" H 4250 5350 50  0001 C CNN
-F 3 "" H 4250 5350 50  0001 C CNN
-	1    4250 5350
-	1    0    0    -1
-$EndComp
-$Comp
-L power:VDDA #PWR0324
-U 1 1 668B4AB2
-P 4650 5350
-F 0 "#PWR0324" H 4650 5200 50  0001 C CNN
-F 1 "VDDA" H 4665 5523 50  0000 C CNN
-F 2 "" H 4650 5350 50  0001 C CNN
-F 3 "" H 4650 5350 50  0001 C CNN
-	1    4650 5350
-	1    0    0    -1
-$EndComp
-$Comp
-L power:VDDA #PWR0329
-U 1 1 668B50B6
-P 5050 5350
-F 0 "#PWR0329" H 5050 5200 50  0001 C CNN
-F 1 "VDDA" H 5065 5523 50  0000 C CNN
-F 2 "" H 5050 5350 50  0001 C CNN
-F 3 "" H 5050 5350 50  0001 C CNN
-	1    5050 5350
 	1    0    0    -1
 $EndComp
@@
 BUSS Voltage Monitor: 0.25x Attenuation
 $Comp
-L power:VPP #PWR?
+L power:VPP #PWR0109
 U 1 1 67282963
 P 4200 4550
-F 0 "#PWR?" H 4200 4400 50  0001 C CNN
+F 0 "#PWR0109" H 4200 4400 50  0001 C CNN
 F 1 "VPP" H 4215 4723 50  0000 C CNN
 F 2 "" H 4200 4550 50  0001 C CNN
@@
 	1    0    0    -1
 $EndComp
+$Comp
+L power:VPP #PWR0113
+U 1 1 64E8D40A
+P 4250 5350
+F 0 "#PWR0113" H 4250 5200 50  0001 C CNN
+F 1 "VPP" H 4265 5523 50  0000 C CNN
+F 2 "" H 4250 5350 50  0001 C CNN
+F 3 "" H 4250 5350 50  0001 C CNN
+	1    4250 5350
+	1    0    0    -1
+$EndComp
