File: flight_computer/v2/microcontroller.sch (KiCad schematic (older format))
At the start: 19 parts, among them U34 MSP430FR5969IRGZR

Commit message: Nearing first pass layout for Rev B flight computer
Parts:
- removed U?: AP2112K-3.3, Package_TO_SOT_SMD:SOT-23-5, symbol Regulator_Linear:AP2112K-3.3
- added C1: 10u, Capacitor_SMD:C_0603_1608Metric, symbol Device:C
- added C111: 0.1u, Capacitor_SMD:C_0603_1608Metric, symbol Device:C
- added C3: 1u, Capacitor_SMD:C_0603_1608Metric, symbol Device:C
- added R1, R2: 4k7, Resistor_SMD:R_0603_1608Metric, symbol Device:R
- added TP1: VREF, TestPoint:TestPoint_Pad_1.0x1.0mm, symbol Connector:TestPoint
- added TP25: 3V3, TestPoint:TestPoint_Pad_1.0x1.0mm, symbol Connector:TestPoint
- added TP26: GND, TestPoint:TestPoint_Pad_1.0x1.0mm, symbol Connector:TestPoint
- C8: renamed from C?; footprint Capacitor_SMD:C_0603_1608Metric -> Capacitor_Tantalum_SMD:CP_EIA-7343-43_Kemet-X
- J1, J2: renamed from J?; footprint (none) -> Connector_Molex:Molex_PicoBlade_53047-0510_1x05_P1.25mm_Vertical
- R57: value R -> 10k
- U7: renamed from U?; footprint TSOT-23_S6_LIT -> Package_TO_SOT_SMD:SOT-23-6
- gave numbers to parts that had none: 3
Connections:
- net 0-9_CLOCK is gone; now on net GAAS_TEMP: U34.35 (P4.6)
- net 10-19_CLOCK is gone; now on net TX_OUT: U34.24 (P2.0/TB0.6/UCA0TXD/UCA0SIMO/TB0CLK/ACLK)
- net ENABLE_PANEL_SWITCH is gone; now on net RX_IN: U34.25 (P2.1/TB0.0/UCA0RXD/UCA0SOMI/TB0.0)
- net +3V3: now also R1.2, R2.2, TP25.1
- net GAAS_TEMP: no longer U34.17 (P4.1/A9)
- net GND: now also C59.2, C1.2, C111.1, C3.2, TP26.1; no longer C59.1
- net LADDER_CLOCK: now also U34.17 (P4.1/A9); no longer U34.10 (P1.4/TB0.1/UCA0STE/A4/C4)
- net RX_IN: no longer U34.21 (P2.6/TB0.1/UCA1RXD/UCA1SOM)
- net SCL: now also U34.32 (P1.7/TB0.4/UCB0SOMI/UCB0SCL/TA1.0), R2.1; no longer U34.31 (P1.6/TB0.3/UCB0SIMO/UCB0SDA/TA0.0)
- net SDA: now also U34.31 (P1.6/TB0.3/UCB0SIMO/UCB0SDA/TA0.0), R1.1; no longer U34.32 (P1.7/TB0.4/UCB0SOMI/UCB0SCL/TA1.0)
- net TX_OUT: no longer U34.20 (P2.5/TB0.0/UCA1TXD/UCA1SIMO)
- net at U34.43 (PJ.7/HFXOUT), Y1.2: now also C59.1; no longer C59.2
- net at U34.2 (P1.1/TA0.2/TA1CLK/COUT/A1/C1/VREF+/VEREF+), U7.6 (VOUT): now also C111.2, TP1.1
- net SET: now reaches U34.26 (P2.2/TB0.2/UCB0CLK)
- net S1_CT: now reaches U34.27 (P3.4/TB0.3/SMCLK)
- net GAAS_ON: now reaches U34.28 (P3.5/TB0.4/COUT)
- net MUX_CLOCK: now reaches U34.29 (P3.6/TB0.5)
- net MAG_INT: now reaches U34.30 (P3.7/TB0.6)
- net BUSY: now reaches U34.33 (P4.4/TB0.5)
- net UNSET: now reaches U34.39 (P2.3/TA0.0/UCA1STE/A6/C10)
- net PANEL_1_ON: now reaches U34.4 (P3.0/A12/C12)
- net VAA: now reaches C60.1, FB2.2, U34.48 (AVCC)
- net VAA: now also C1.1, C3.1
- net PANEL_2_ON: now reaches U34.5 (P3.1/A13/C13)
- net PANEL_3_ON: now reaches U34.6 (P3.2/A14/C14)
- net S0_CT: now reaches U34.7 (P3.3/A15/C15)
- net CT_GOOD: now reaches U34.8 (P4.7)
- net ALERT renamed READ_BUSS
- net ENABLE_TEST_SOURCE renamed TRACE_DIR
- net LADDER_LATCH renamed NO_V
- net RESET_PANEL_SWITCH renamed MUX_GOOD
- net ~LADDER_EN renamed NC_V
- net ~LADDER_RESET renamed READ_VOLTAGE
- new net READ_CURRENT: U34.10 (P1.4/TB0.1/UCA0STE/A4/C4)
- new net RX: U34.21 (P2.6/TB0.1/UCA1RXD/UCA1SOM)
- new net TX: U34.20 (P2.5/TB0.0/UCA1TXD/UCA1SIMO)
- no-connect marks 10 -> 5
Other:
- moved on the sheet: C10, C11, C12, C13, C2, C4, C5, C6, C7, C8, C9, FB1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

Commit message: Finished layout of flight computer
Parts:
- added C18: 0.1u, Capacitor_SMD:C_0603_1608Metric, symbol Device:C
Connections:
- net PANEL_1_ON is gone; now on net NO_V: U34.4 (P3.0/A12/C12)
- net PANEL_2_ON is gone; now on net UNSET: U34.5 (P3.1/A13/C13)
- net +3V3: now also C18.2
- net BUSY: now also U34.34 (P4.5); no longer U34.33 (P4.4/TB0.5)
- net CT_GOOD: now also U34.27 (P3.4/TB0.3/SMCLK); no longer U34.8 (P4.7)
- net GAAS_TEMP: now also U34.33 (P4.4/TB0.5); no longer U34.35 (P4.6)
- net GND: now also C18.1
- net MAG_INT: now also U34.7 (P3.3/A15/C15); no longer U34.30 (P3.7/TB0.6)
- net MUX_CLOCK: now also U34.30 (P3.7/TB0.6); no longer U34.29 (P3.6/TB0.5)
- net MUX_GOOD: now also U34.29 (P3.6/TB0.5); no longer U34.34 (P4.5)
- net NO_V: no longer U34.9 (P1.3/TA1.2/UCB0STE/A3/C3)
- net PANEL_3_ON: now also U34.35 (P4.6); no longer U34.6 (P3.2/A14/C14)
- net PAYLOAD_RST: now also J2.4 (Pin_4); no longer J1.3 (Pin_3)
- net RX_IN: now also J1.2 (Pin_2); no longer J2.3 (Pin_3)
- net S0_CT: now also U34.8 (P4.7); no longer U34.7 (P3.3/A15/C15)
- net S1_CT: now also U34.9 (P1.3/TA1.2/UCB0STE/A3/C3); no longer U34.27 (P3.4/TB0.3/SMCLK)
- net SET: now also U34.6 (P3.2/A14/C14); no longer U34.26 (P2.2/TB0.2/UCB0CLK)
- net TEST: now also J2.3 (Pin_3); no longer J1.2 (Pin_2)
- net TX_OUT: now also J1.3 (Pin_3); no longer J2.4 (Pin_4)
- net UNSET: no longer U34.39 (P2.3/TA0.0/UCA1STE/A6/C10)
- no-connect marks 5 -> 7
Changed lines of the file:
@@
 $Descr A4 11693 8268
 encoding utf-8
-Sheet 2 8
+Sheet 8 8
 Title "Radiation Hardened Microcontroller Circuits"
 Date "2023-08-13"
@@
 Wire Wire Line
 	2800 2100 3150 2100
+Text GLabel 950  7250 2    50   Input ~ 0
+PAYLOAD_RST
+Text GLabel 950  6350 2    50   Input ~ 0
+RX_IN
 Text GLabel 950  6450 2    50   Input ~ 0
-PAYLOAD_RST
-Text GLabel 950  7150 2    50   Input ~ 0
-RX_IN
-Text GLabel 950  7250 2    50   Input ~ 0
 TX_OUT
 $Comp
@@
 Wire Wire Line
 	1050 7350 1050 7450
-Text GLabel 950  6350 2    50   Input ~ 0
-TEST
 Text GLabel 950  7050 2    50   Input ~ 0
 TCK
@@
 Text HLabel 4250 3550 0    50   Input ~ 0
 READ_VOLTAGE
-Text HLabel 7300 3350 2    50   Input ~ 0
+Text HLabel 7300 4550 2    50   Input ~ 0
 S0_CT
-Text HLabel 7300 3450 2    50   Input ~ 0
+Text HLabel 4250 3350 0    50   Input ~ 0
 S1_CT
 Text HLabel 7300 3550 2    50   Input ~ 0
 GAAS_ON
+Text HLabel 7300 3750 2    50   Input ~ 0
+MUX_CLOCK
 Text HLabel 7300 3650 2    50   Input ~ 0
-MUX_CLOCK
-Text HLabel 7300 4350 2    50   Input ~ 0
 MUX_GOOD
-Text HLabel 7300 4450 2    50   Input ~ 0
+Text HLabel 7300 4250 2    50   Input ~ 0
 GAAS_TEMP
 Text HLabel 7300 3950 2    50   Input ~ 0
@@
 Text HLabel 7300 4050 2    50   Input ~ 0
 TRACE_DIR
-Text HLabel 7300 4550 2    50   Input ~ 0
+Text HLabel 7300 3450 2    50   Input ~ 0
 CT_GOOD
-Text HLabel 7300 3050 2    50   Input ~ 0
-PANEL_1_ON
-Text HLabel 7300 3150 2    50   Input ~ 0
-PANEL_2_ON
-Text HLabel 7300 3250 2    50   Input ~ 0
+Text HLabel 7300 4450 2    50   Input ~ 0
 PANEL_3_ON
 Text HLabel 2650 4450 0    50   Input ~ 0
@@
 Text HLabel 2650 4350 0    50   Input ~ 0
 SDA
-Text HLabel 7300 4250 2    50   Input ~ 0
+Text HLabel 7300 4350 2    50   Input ~ 0
 BUSY
 Text HLabel 4250 4450 0    50   Input ~ 0
@@
 Text HLabel 4250 4350 0    50   Input ~ 0
 TX
-Text HLabel 7300 3750 2    50   Input ~ 0
+Text HLabel 7300 3350 2    50   Input ~ 0
 MAG_INT
-Text HLabel 4250 4050 0    50   Input ~ 0
+Text HLabel 7300 3250 2    50   Input ~ 0
 SET
-Text HLabel 4250 4150 0    50   Input ~ 0
+Text HLabel 7300 3150 2    50   Input ~ 0
 UNSET
-Text HLabel 4250 3350 0    50   Input ~ 0
+Text HLabel 7300 3050 2    50   Input ~ 0
 NO_V
 Text HLabel 4250 3250 0    50   Input ~ 0
@@
 Wire Wire Line
 	1250 3050 4250 3050
+$Comp
+L Device:C C?
+U 1 1 6513B657
+P 2050 7200
+AR Path="/6313FC31/6513B657" Ref="C?"  Part="1"
+AR Path="/6513B657" Ref="C?"  Part="1"
+AR Path="/635FE71D/6513B657" Ref="C?"  Part="1"
+AR Path="/63D1F518/6513B657" Ref="C?"  Part="1"
+AR Path="/63D21EEE/6513B657" Ref="C?"  Part="1"
+AR Path="/64AE160A/6513B657" Ref="C18"  Part="1"
+F 0 "C18" V 2302 7200 50  0000 C CNN
+F 1 "0.1u" V 2211 7200 50  0000 C CNN
+F 2 "Capacitor_SMD:C_0603_1608Metric" H 2088 7050 50  0001 C CNN
+F 3 "~" H 2050 7200 50  0001 C CNN
+	1    2050 7200
+	-1   0    0    1
+$EndComp
+$Comp
+L power:GND #PWR?
+U 1 1 6513B65D
+P 2050 7350
+AR Path="/6313FC31/6513B65D" Ref="#PWR?"  Part="1"
+AR Path="/6513B65D" Ref="#PWR?"  Part="1"
+AR Path="/635FE71D/6513B65D" Ref="#PWR?"  Part="1"
+AR Path="/63D1F518/6513B65D" Ref="#PWR?"  Part="1"
+AR Path="/63D21EEE/6513B65D" Ref="#PWR?"  Part="1"
+AR Path="/64AE160A/6513B65D" Ref="#PWR0154"  Part="1"
+F 0 "#PWR0154" H 2050 7100 50  0001 C CNN
+F 1 "GND" H 2055 7177 50  0000 C CNN
+F 2 "" H 2050 7350 50  0001 C CNN
+F 3 "" H 2050 7350 50  0001 C CNN
+	1    2050 7350
+	1    0    0    -1
+$EndComp
+$Comp
+L power:+3V3 #PWR?
+U 1 1 6513C640
+P 2050 7050
+AR Path="/6513C640" Ref="#PWR?"  Part="1"
+AR Path="/63D1F518/6513C640" Ref="#PWR?"  Part="1"
+AR Path="/63D21EEE/6513C640" Ref="#PWR?"  Part="1"
+AR Path="/64AE160A/6513C640" Ref="#PWR0158"  Part="1"
+F 0 "#PWR0158" H 2050 6900 50  0001 C CNN
+F 1 "+3V3" H 2065 7223 50  0000 C CNN
+F 2 "" H 2050 7050 50  0001 C CNN
+F 3 "" H 2050 7050 50  0001 C CNN
+	1    2050 7050
+	1    0    0    -1
+$EndComp
+Text GLabel 950  7150 2    50   Input ~ 0
+TEST
+NoConn ~ 4250 4050
+NoConn ~ 4250 4150
 $EndSCHEMATC
