File: flight_computer/v2/switcher.sch (KiCad schematic (older format))
At the start: 56 parts, among them J10 Perovskite 3, J11 GaAs Panel, J12 GaAs Temperature, J13 Perovskite 1, J14 Perovskite 2, U2 CD4518BM96, U39 74AHC1G08, U40 CD4514BM, U41 CD4514BM, U42 ADG839YKSZ-REEL7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

Commit message: Finished layout of flight computer
Parts:
- removed C22, C94, C95, C98: 0.1u, Capacitor_SMD:C_0603_1608Metric, symbol Device:C
- added C17, C28, C29: 0.1u, Capacitor_SMD:C_0603_1608Metric, symbol Device:C
Connections:
- net GND: now also C17.2, C28.2, C29.2
- net VBUS: now also C17.1, C28.1, C29.1
- net P1_P1: now reaches J13.6 (Pin_6), U47.5 (D)
- net P1_P6: now reaches J13.3 (Pin_3), U44.5 (D)
- net P1_P3: now reaches J13.4 (Pin_4), U45.5 (D)
- net P1_P4: now reaches U43.5 (D)
- net P1_P4: now also J13.1 (Pin_1); no longer J13.2 (Pin_2)
- net P1_P2: now reaches J13.5 (Pin_5), U46.5 (D)
- net P1_P5: now reaches U42.5 (D)
- net P1_P5: now also J13.2 (Pin_2); no longer J13.1 (Pin_1)
- net P2_P1: now reaches J14.6 (Pin_6)
- net P2_P1: now also U52.5 (D); no longer U53.5 (D)
- net P2_P6: now reaches J14.3 (Pin_3), U50.5 (D)
- net P2_P3: now reaches U49.5 (D)
- net P2_P3: now also J14.4 (Pin_4); no longer J14.2 (Pin_2)
- net P2_P4: now reaches J14.1 (Pin_1), U48.5 (D)
- net P2_P2: now reaches J14.5 (Pin_5)
- net P2_P2: now also U53.5 (D); no longer U52.5 (D)
- net P2_P5: now reaches U51.5 (D)
- net P2_P5: now also J14.2 (Pin_2); no longer J14.4 (Pin_4)
- net P3_P1: now reaches J10.6 (Pin_6), U59.5 (D)
- net P3_P6: now reaches J10.3 (Pin_3), U56.5 (D)
- net P3_P5: now reaches J10.2 (Pin_2), U55.5 (D)
- net P3_P4: now reaches J10.1 (Pin_1), U54.5 (D)
- net P3_P2: now reaches J10.5 (Pin_5), U58.5 (D)
- net P3_P3: now reaches J10.4 (Pin_4), U57.5 (D)
- net PEROVSKITE_1_POS renamed P1_CP
- net PEROVSKITE_2_POS renamed P2_CP
- net PEROVSKITE_3_POS renamed P3_CP
Other:
- moved on the sheet: C83, J10, J13, J14
