File: flight_computer/v2/resistor_ladder.sch (KiCad schematic (older format))
At the start: 58 parts, among them U18 ADG841YKSZ-500RL7, U19 ADG841YKSZ-500RL7, U20 ADG841YKSZ-500RL7, U21 CD4516B_PW_16, U22 ADG841YKSZ-500RL7, U26 CD4516B_PW_16, U28 ADG841YKSZ-500RL7, U29 ADG841YKSZ-500RL7, U30 ADG841YKSZ-500RL7, U31 CD4516B_PW_16, U32 ADG841YKSZ-500RL7, U33 ADG841YKSZ-500RL7, U34 ADG841YKSZ-500RL7, U35 ADG841YKSZ-500RL7, U36 CD4516B_PW_16, U37 ADG841YKSZ-500RL7, U6 4012, U6 ADG841YKSZ-500RL7, U7 ADG841YKSZ-500RL7, U8 ADG841YKSZ-500RL7, U9 ADG841YKSZ-500RL7

Commit message: Finishing touches
- Fill out bill of material
- Add selection guides
- Update curve tracer resistors
- Update finish date
Parts:
- R55, R59, R63, R67: value 1M -> 120
- R56, R60, R64, R68: value 250 -> 270
- R57, R61, R65, R69: value 500 -> 430
Changed lines of the file:
@@
 P 5300 3350
 F 0 "R59" V 5093 3350 50  0000 C CNN
-F 1 "1M" V 5184 3350 50  0000 C CNN
+F 1 "120" V 5184 3350 50  0000 C CNN
 F 2 "Resistor_SMD:R_0603_1608Metric" V 5230 3350 50  0001 C CNN
 F 3 "~" H 5300 3350 50  0001 C CNN
@@
 P 5950 3350
 F 0 "R60" V 5743 3350 50  0000 C CNN
-F 1 "250" V 5834 3350 50  0000 C CNN
+F 1 "270" V 5834 3350 50  0000 C CNN
 F 2 "Resistor_SMD:R_0603_1608Metric" V 5880 3350 50  0001 C CNN
 F 3 "~" H 5950 3350 50  0001 C CNN
@@
 P 6600 3350
 F 0 "R61" V 6393 3350 50  0000 C CNN
-F 1 "500" V 6484 3350 50  0000 C CNN
+F 1 "430" V 6484 3350 50  0000 C CNN
 F 2 "Resistor_SMD:R_0603_1608Metric" V 6530 3350 50  0001 C CNN
 F 3 "~" H 6600 3350 50  0001 C CNN
@@
 P 8800 3350
 F 0 "R63" V 8593 3350 50  0000 C CNN
-F 1 "1M" V 8684 3350 50  0000 C CNN
+F 1 "120" V 8684 3350 50  0000 C CNN
 F 2 "Resistor_SMD:R_0603_1608Metric" V 8730 3350 50  0001 C CNN
 F 3 "~" H 8800 3350 50  0001 C CNN
@@
 P 9450 3350
 F 0 "R64" V 9243 3350 50  0000 C CNN
-F 1 "250" V 9334 3350 50  0000 C CNN
+F 1 "270" V 9334 3350 50  0000 C CNN
 F 2 "Resistor_SMD:R_0603_1608Metric" V 9380 3350 50  0001 C CNN
 F 3 "~" H 9450 3350 50  0001 C CNN
@@
 P 10100 3350
 F 0 "R65" V 9893 3350 50  0000 C CNN
-F 1 "500" V 9984 3350 50  0000 C CNN
+F 1 "430" V 9984 3350 50  0000 C CNN
 F 2 "Resistor_SMD:R_0603_1608Metric" V 10030 3350 50  0001 C CNN
 F 3 "~" H 10100 3350 50  0001 C CNN
@@
 P 1800 3350
 F 0 "R55" V 1593 3350 50  0000 C CNN
-F 1 "1M" V 1684 3350 50  0000 C CNN
+F 1 "120" V 1684 3350 50  0000 C CNN
 F 2 "Resistor_SMD:R_0603_1608Metric" V 1730 3350 50  0001 C CNN
 F 3 "~" H 1800 3350 50  0001 C CNN
@@
 P 2450 3350
 F 0 "R56" V 2243 3350 50  0000 C CNN
-F 1 "250" V 2334 3350 50  0000 C CNN
+F 1 "270" V 2334 3350 50  0000 C CNN
 F 2 "Resistor_SMD:R_0603_1608Metric" V 2380 3350 50  0001 C CNN
 F 3 "~" H 2450 3350 50  0001 C CNN
@@
 P 3100 3350
 F 0 "R57" V 2893 3350 50  0000 C CNN
-F 1 "500" V 2984 3350 50  0000 C CNN
+F 1 "430" V 2984 3350 50  0000 C CNN
 F 2 "Resistor_SMD:R_0603_1608Metric" V 3030 3350 50  0001 C CNN
 F 3 "~" H 3100 3350 50  0001 C CNN
@@
 P 12400 3350
 F 0 "R67" V 12193 3350 50  0000 C CNN
-F 1 "1M" V 12284 3350 50  0000 C CNN
+F 1 "120" V 12284 3350 50  0000 C CNN
 F 2 "Resistor_SMD:R_0603_1608Metric" V 12330 3350 50  0001 C CNN
 F 3 "~" H 12400 3350 50  0001 C CNN
@@
 P 13050 3350
 F 0 "R68" V 12843 3350 50  0000 C CNN
-F 1 "250" V 12934 3350 50  0000 C CNN
+F 1 "270" V 12934 3350 50  0000 C CNN
 F 2 "Resistor_SMD:R_0603_1608Metric" V 12980 3350 50  0001 C CNN
 F 3 "~" H 13050 3350 50  0001 C CNN
@@
 P 13700 3350
 F 0 "R69" V 13493 3350 50  0000 C CNN
-F 1 "500" V 13584 3350 50  0000 C CNN
+F 1 "430" V 13584 3350 50  0000 C CNN
 F 2 "Resistor_SMD:R_0603_1608Metric" V 13630 3350 50  0001 C CNN
 F 3 "~" H 13700 3350 50  0001 C CNN

Commit message: Create v3 flight computer
Parts:
- added unit 2 of U6
Connections:
- net GND: now also U21.12 (P2), U21.13 (P3), U21.3 (P4), U21.4 (P1), U21.5 (*CARRYIN), U26.12 (P2), U26.13 (P3), U26.3 (P4), U26.4 (P1), U26.5 (*CARRYIN), U31.12 (P2), U31.13 (P3), U31.3 (P4), U31.4 (P1), U31.5 (*CARRYIN), U36.12 (P2), U36.13 (P3), U36.3 (P4), U36.4 (P1), U36.5 (*CARRYIN), U6.10, U6.11, U6.12, U6.9
- no-connect marks 24 -> 5
Changed lines of the file:
@@
 Date "2023-08-16"
 Rev "C"
-Comp "UNL Aerospace Club | Advanced eXperimental Payloads"
+Comp "UNL Aerospace Club | Aerospace eXperimental Payloads"
 Comment1 "Copyright (c) 2023"
 Comment2 "Designer: WSA"
@@
 $EndComp
 $Comp
-L CD4516BPWR:CD4516B_PW_16 U26
-U 1 1 64EB28CD
-P 7250 6600
-F 0 "U26" H 7275 7287 60  0000 C CNN
-F 1 "CD4516B_PW_16" H 7275 7181 60  0000 C CNN
-F 2 "Package_SO:TSSOP-16_4.4x5mm_P0.65mm" H 7250 7190 60  0001 C CNN
-F 3 "" H 6400 6950 60  0000 C CNN
-	1    7250 6600
-	0    -1   -1   0
-$EndComp
-$Comp
 L power:GND #PWR0197
 U 1 1 63350ACA
@@
 	1    0    0    -1
 $EndComp
-NoConn ~ 7100 7450
-NoConn ~ 7200 7450
-NoConn ~ 7300 7450
-NoConn ~ 7400 7450
-NoConn ~ 7600 5700
-NoConn ~ 7500 5700
 $Comp
 L power:GND #PWR0200
@@
 	1    0    0    -1
 $EndComp
-NoConn ~ 10600 7450
-NoConn ~ 10700 7450
-NoConn ~ 10800 7450
-NoConn ~ 10900 7450
 NoConn ~ 11100 5700
-NoConn ~ 11000 5700
 $Comp
 L power:GND #PWR0207
@@
 	3950 3650 3950 3350
 $Comp
-L CD4516BPWR:CD4516B_PW_16 U21
-U 1 1 65CDCBD2
-P 3750 6600
-F 0 "U21" H 3775 7287 60  0000 C CNN
-F 1 "CD4516B_PW_16" H 3775 7181 60  0000 C CNN
-F 2 "Package_SO:TSSOP-16_4.4x5mm_P0.65mm" H 3750 7190 60  0001 C CNN
-F 3 "" H 2900 6950 60  0000 C CNN
-	1    3750 6600
-	0    -1   -1   0
-$EndComp
-$Comp
 L power:GND #PWR0178
 U 1 1 65CDCBDF
@@
 	1    0    0    -1
 $EndComp
-NoConn ~ 3600 7450
-NoConn ~ 3700 7450
-NoConn ~ 3800 7450
-NoConn ~ 3900 7450
 NoConn ~ 4100 5700
-NoConn ~ 4000 5700
 $Comp
 L power:GND #PWR0181
@@
 	1    0    0    -1
 $EndComp
-NoConn ~ 14200 7450
-NoConn ~ 14300 7450
-NoConn ~ 14400 7450
-NoConn ~ 14500 7450
 NoConn ~ 14700 5700
-NoConn ~ 14600 5700
 $Comp
 L power:GND #PWR0212
@@
 	10400 7750 10400 7450
 Wire Wire Line
-	10400 7750 14000 7750
+	10400 7750 10600 7750
 Wire Wire Line
 	14000 7750 14000 7450
@@
 	4300 5600 4300 5700
 Wire Wire Line
-	3500 5600 4300 5600
+	3500 5600 4000 5600
 Wire Wire Line
 	7000 5700 7000 5600
 Wire Wire Line
-	7000 5600 7800 5600
+	7000 5600 7500 5600
 Wire Wire Line
 	7800 5600 7800 5700
@@
 	10500 5700 10500 5600
 Wire Wire Line
-	10500 5600 11350 5600
+	10500 5600 11000 5600
 Wire Wire Line
 	11350 5600 11350 5700
@@
 	14100 5700 14100 5600
 Wire Wire Line
-	14100 5600 14950 5600
+	14100 5600 14600 5600
 Wire Wire Line
 	14950 5600 14950 5700
@@
 Connection ~ 6900 7750
 Wire Wire Line
-	6900 7750 10400 7750
+	6900 7750 7100 7750
 Connection ~ 7000 7850
 Wire Wire Line
@@
 	7500 7950 11000 7950
 Wire Wire Line
-	3400 7750 6900 7750
+	3400 7750 3600 7750
 Wire Wire Line
 	3500 7850 7000 7850
@@
 	1    0    0    -1
 $EndComp
+NoConn ~ 7600 5700
+Wire Wire Line
+	11000 5700 11000 5600
+Connection ~ 11000 5600
+Wire Wire Line
+	11000 5600 11350 5600
+Wire Wire Line
+	7500 5700 7500 5600
+Connection ~ 7500 5600
+Wire Wire Line
+	7500 5600 7800 5600
+$Comp
+L CD4516BPWR:CD4516B_PW_16 U21
+U 1 1 65CDCBD2
+P 3750 6600
+F 0 "U21" H 3775 7287 60  0000 C CNN
+F 1 "CD4516B_PW_16" H 3775 7181 60  0000 C CNN
+F 2 "Package_SO:TSSOP-16_4.4x5mm_P0.65mm" H 3750 7190 60  0001 C CNN
+F 3 "" H 2900 6950 60  0000 C CNN
+	1    3750 6600
+	0    -1   -1   0
+$EndComp
+Wire Wire Line
+	4000 5700 4000 5600
+Connection ~ 4000 5600
+Wire Wire Line
+	4000 5600 4300 5600
+Wire Wire Line
+	14600 5700 14600 5600
+Connection ~ 14600 5600
+Wire Wire Line
+	14600 5600 14950 5600
+$Comp
+L CD4516BPWR:CD4516B_PW_16 U26
+U 1 1 64EB28CD
+P 7250 6600
+F 0 "U26" H 7275 7287 60  0000 C CNN
+F 1 "CD4516B_PW_16" H 7275 7181 60  0000 C CNN
+F 2 "Package_SO:TSSOP-16_4.4x5mm_P0.65mm" H 7250 7190 60  0001 C CNN
+F 3 "" H 6400 6950 60  0000 C CNN
+	1    7250 6600
+	0    -1   -1   0
+$EndComp
+Wire Wire Line
+	3600 7450 3600 7750
+Connection ~ 3600 7750
+Wire Wire Line
+	3600 7750 3700 7750
+Wire Wire Line
+	3700 7450 3700 7750
+Connection ~ 3700 7750
+Wire Wire Line
+	3700 7750 3800 7750
+Wire Wire Line
+	3800 7450 3800 7750
+Connection ~ 3800 7750
+Wire Wire Line
+	3800 7750 3900 7750
+Wire Wire Line
+	3900 7450 3900 7750
+Connection ~ 3900 7750
+Wire Wire Line
+	3900 7750 6900 7750
+Wire Wire Line
+	7100 7450 7100 7750
+Connection ~ 7100 7750
+Wire Wire Line
+	7100 7750 7200 7750
+Wire Wire Line
+	7200 7750 7200 7450
+Connection ~ 7200 7750
+Wire Wire Line
+	7200 7750 7300 7750
+Wire Wire Line
+	7300 7450 7300 7750
+Connection ~ 7300 7750
+Wire Wire Line
+	7300 7750 7400 7750
+Wire Wire Line
+	7400 7750 7400 7450
+Connection ~ 7400 7750
+Wire Wire Line
+	7400 7750 10400 7750
+Wire Wire Line
+	10600 7450 10600 7750
+Connection ~ 10600 7750
+Wire Wire Line
+	10600 7750 10700 7750
+Wire Wire Line
+	10700 7750 10700 7450
+Connection ~ 10700 7750
+Wire Wire Line
+	10800 7450 10800 7750
+Wire Wire Line
+	10700 7750 10800 7750
+Connection ~ 10800 7750
+Wire Wire Line
+	10800 7750 10900 7750
+Wire Wire Line
+	10900 7750 10900 7450
+Connection ~ 10900 7750
+Wire Wire Line
+	10900 7750 14000 7750
+Wire Wire Line
+	14000 7750 14200 7750
+Wire Wire Line
+	14500 7750 14500 7450
+Connection ~ 14000 7750
+Wire Wire Line
+	14400 7450 14400 7750
+Connection ~ 14400 7750
+Wire Wire Line
+	14400 7750 14500 7750
+Wire Wire Line
+	14300 7450 14300 7750
+Connection ~ 14300 7750
+Wire Wire Line
+	14300 7750 14400 7750
+Wire Wire Line
+	14200 7450 14200 7750
+Connection ~ 14200 7750
+Wire Wire Line
+	14200 7750 14300 7750
+$Comp
+L 4xxx:4012 U6
+U 2 1 650E82D8
+P 3200 9100
+F 0 "U6" H 3200 8758 50  0000 C CNN
+F 1 "4012" H 3200 8849 50  0000 C CNN
+F 2 "Package_SO:TSSOP-14_4.4x5mm_P0.65mm" H 3200 9100 50  0001 C CNN
+F 3 "http://www.intersil.com/content/dam/Intersil/documents/cd40/cd4011bms-12bms-23bms.pdf" H 3200 9100 50  0001 C CNN
+	2    3200 9100
+	-1   0    0    1
+$EndComp
+$Comp
+L power:GND #PWR0162
+U 1 1 650ECA30
+P 3600 9350
+F 0 "#PWR0162" H 3600 9100 50  0001 C CNN
+F 1 "GND" H 3605 9177 50  0000 C CNN
+F 2 "" H 3600 9350 50  0001 C CNN
+F 3 "" H 3600 9350 50  0001 C CNN
+	1    3600 9350
+	1    0    0    -1
+$EndComp
+Wire Wire Line
+	3500 8950 3600 8950
+Wire Wire Line
+	3600 8950 3600 9050
+Wire Wire Line
+	3500 9250 3600 9250
+Connection ~ 3600 9250
+Wire Wire Line
+	3600 9250 3600 9350
+Connection ~ 3600 9150
+Wire Wire Line
+	3600 9150 3600 9250
+Wire Wire Line
+	3500 9050 3600 9050
+Connection ~ 3600 9050
+Wire Wire Line
+	3600 9050 3600 9150
+Wire Wire Line
+	3500 9150 3600 9150
+NoConn ~ 2900 9100
 $EndSCHEMATC
