File: secondary_payload/brs_flight_computer.sch (KiCad schematic (older format))
At the start: 6 parts, among them J1 Conn_01x06_Male, J2 Conn_01x06_Male, J3 Conn_01x10_Male, J4 Conn_01x16_Male, J5 Conn_01x03_Male, J6 Conn_01x12_Male

Commit message: Updating based on harnesses
Parts:
- added J7, J8: Conn_01x06_Male, Connector_PinHeader_2.54mm:PinHeader_1x06_P2.54mm_Vertical, symbol Connector:Conn_01x06_Male
Connections:
- net GND: now also J7.4 (Pin_4)
- net SCL: now also J7.3 (Pin_3)
- net SDA: now also J7.2 (Pin_2)
- net VDDF: now also J7.6 (Pin_6)
- no-connect marks 7 -> 15
Changed lines of the file:
@@
 	-1   0    0    1
 $EndComp
+$Comp
+L Connector:Conn_01x06_Male J7
+U 1 1 64F13341
+P 4100 5150
+F 0 "J7" H 4072 5078 50  0000 R CNN
+F 1 "Conn_01x06_Male" H 4072 5123 50  0001 R CNN
+F 2 "Connector_PinHeader_2.54mm:PinHeader_1x06_P2.54mm_Vertical" H 4100 5150 50  0001 C CNN
+F 3 "~" H 4100 5150 50  0001 C CNN
+	1    4100 5150
+	-1   0    0    1
+$EndComp
+$Comp
+L Connector:Conn_01x06_Male J8
+U 1 1 64F13347
+P 4350 5050
+F 0 "J8" H 4458 5339 50  0000 C CNN
+F 1 "Conn_01x06_Male" H 4458 5340 50  0001 C CNN
+F 2 "Connector_PinHeader_2.54mm:PinHeader_1x06_P2.54mm_Vertical" H 4350 5050 50  0001 C CNN
+F 3 "~" H 4350 5050 50  0001 C CNN
+	1    4350 5050
+	1    0    0    -1
+$EndComp
+$Comp
+L power:VDDF #PWR?
+U 1 1 64F1334D
+P 3800 4800
+AR Path="/64D821F3/64F1334D" Ref="#PWR?"  Part="1"
+AR Path="/6685FD81/64F1334D" Ref="#PWR?"  Part="1"
+AR Path="/64F1334D" Ref="#PWR0109"  Part="1"
+F 0 "#PWR0109" H 3800 4650 50  0001 C CNN
+F 1 "VDDF" H 3815 4973 50  0000 C CNN
+F 2 "" H 3800 4800 50  0001 C CNN
+F 3 "" H 3800 4800 50  0001 C CNN
+	1    3800 4800
+	1    0    0    -1
+$EndComp
+$Comp
+L power:GND #PWR?
+U 1 1 64F13353
+P 3900 5050
+AR Path="/6685FD81/64F13353" Ref="#PWR?"  Part="1"
+AR Path="/64F13353" Ref="#PWR0110"  Part="1"
+F 0 "#PWR0110" H 3900 4800 50  0001 C CNN
+F 1 "GND" V 3905 4922 50  0000 R CNN
+F 2 "" H 3900 5050 50  0001 C CNN
+F 3 "" H 3900 5050 50  0001 C CNN
+	1    3900 5050
+	0    1    1    0
+$EndComp
+Text HLabel 3900 5150 0    50   Input ~ 0
+SCL
+Text HLabel 3900 5250 0    50   Input ~ 0
+SDA
+Wire Wire Line
+	3900 4850 3800 4850
+Wire Wire Line
+	3800 4850 3800 4800
+NoConn ~ 3900 4950
+NoConn ~ 4550 4850
+NoConn ~ 4550 4950
+NoConn ~ 4550 5050
+NoConn ~ 4550 5150
+NoConn ~ 4550 5250
+NoConn ~ 4550 5350
+NoConn ~ 3900 5350
 $EndSCHEMATC

Commit message: Integrating flight computer
- EPS commands tested and working
- Updated v3, fixing connector polarity
Parts:
- added C1, C2: C, Capacitor_THT:C_Disc_D5.0mm_W2.5mm_P5.00mm, symbol Device:C
- added R1, R2: R, Resistor_THT:R_Axial_DIN0207_L6.3mm_D2.5mm_P15.24mm_Horizontal, symbol Device:R
Connections:
- net GND: now also C1.2, C2.2, R1.2, R2.2
- net NC_V: now also C1.1, R1.1
- net NO_V: now also C2.1, R2.1
Changed lines of the file:
@@
 	0    1    1    0
 $EndComp
-Text HLabel 8250 4850 3    50   Input ~ 0
+Text HLabel 9200 4950 2    50   Input ~ 0
 NO_V
-Text HLabel 8050 4850 3    50   Input ~ 0
+Text HLabel 7100 4950 0    50   Input ~ 0
 NC_V
 $Comp
@@
 NoConn ~ 4550 5350
 NoConn ~ 3900 5350
+$Comp
+L Device:C C1
+U 1 1 64F4BFC0
+P 7550 5200
+F 0 "C1" H 7665 5246 50  0000 L CNN
+F 1 "C" H 7665 5155 50  0000 L CNN
+F 2 "Capacitor_THT:C_Disc_D5.0mm_W2.5mm_P5.00mm" H 7588 5050 50  0001 C CNN
+F 3 "~" H 7550 5200 50  0001 C CNN
+	1    7550 5200
+	1    0    0    -1
+$EndComp
+$Comp
+L Device:R R1
+U 1 1 64F4C7BF
+P 7300 5200
+F 0 "R1" H 7370 5246 50  0000 L CNN
+F 1 "R" H 7370 5155 50  0000 L CNN
+F 2 "Resistor_THT:R_Axial_DIN0207_L6.3mm_D2.5mm_P15.24mm_Horizontal" V 7230 5200 50  0001 C CNN
+F 3 "~" H 7300 5200 50  0001 C CNN
+	1    7300 5200
+	1    0    0    -1
+$EndComp
+$Comp
+L power:GND #PWR?
+U 1 1 64F4CFAD
+P 7300 5350
+AR Path="/6685FD81/64F4CFAD" Ref="#PWR?"  Part="1"
+AR Path="/64F4CFAD" Ref="#PWR0111"  Part="1"
+F 0 "#PWR0111" H 7300 5100 50  0001 C CNN
+F 1 "GND" V 7305 5222 50  0000 R CNN
+F 2 "" H 7300 5350 50  0001 C CNN
+F 3 "" H 7300 5350 50  0001 C CNN
+	1    7300 5350
+	1    0    0    -1
+$EndComp
+$Comp
+L power:GND #PWR?
+U 1 1 64F4DA93
+P 7550 5350
+AR Path="/6685FD81/64F4DA93" Ref="#PWR?"  Part="1"
+AR Path="/64F4DA93" Ref="#PWR0112"  Part="1"
+F 0 "#PWR0112" H 7550 5100 50  0001 C CNN
+F 1 "GND" V 7555 5222 50  0000 R CNN
+F 2 "" H 7550 5350 50  0001 C CNN
+F 3 "" H 7550 5350 50  0001 C CNN
+	1    7550 5350
+	1    0    0    -1
+$EndComp
+Wire Wire Line
+	8050 4850 8050 4950
+Wire Wire Line
+	8050 4950 7550 4950
+Wire Wire Line
+	7300 5050 7300 4950
+Connection ~ 7300 4950
+Wire Wire Line
+	7300 4950 7100 4950
+Wire Wire Line
+	7550 5050 7550 4950
+Connection ~ 7550 4950
+Wire Wire Line
+	7550 4950 7300 4950
+$Comp
+L Device:C C2
+U 1 1 64F4F9AB
+P 9050 5200
+F 0 "C2" H 9165 5246 50  0000 L CNN
+F 1 "C" H 9165 5155 50  0000 L CNN
+F 2 "Capacitor_THT:C_Disc_D5.0mm_W2.5mm_P5.00mm" H 9088 5050 50  0001 C CNN
+F 3 "~" H 9050 5200 50  0001 C CNN
+	1    9050 5200
+	1    0    0    -1
+$EndComp
+$Comp
+L Device:R R2
+U 1 1 64F4F9B1
+P 8800 5200
+F 0 "R2" H 8870 5246 50  0000 L CNN
+F 1 "R" H 8870 5155 50  0000 L CNN
+F 2 "Resistor_THT:R_Axial_DIN0207_L6.3mm_D2.5mm_P15.24mm_Horizontal" V 8730 5200 50  0001 C CNN
+F 3 "~" H 8800 5200 50  0001 C CNN
+	1    8800 5200
+	1    0    0    -1
+$EndComp
+$Comp
+L power:GND #PWR?
+U 1 1 64F4F9B7
+P 8800 5350
+AR Path="/6685FD81/64F4F9B7" Ref="#PWR?"  Part="1"
+AR Path="/64F4F9B7" Ref="#PWR0113"  Part="1"
+F 0 "#PWR0113" H 8800 5100 50  0001 C CNN
+F 1 "GND" V 8805 5222 50  0000 R CNN
+F 2 "" H 8800 5350 50  0001 C CNN
+F 3 "" H 8800 5350 50  0001 C CNN
+	1    8800 5350
+	1    0    0    -1
+$EndComp
+$Comp
+L power:GND #PWR?
+U 1 1 64F4F9BD
+P 9050 5350
+AR Path="/6685FD81/64F4F9BD" Ref="#PWR?"  Part="1"
+AR Path="/64F4F9BD" Ref="#PWR0114"  Part="1"
+F 0 "#PWR0114" H 9050 5100 50  0001 C CNN
+F 1 "GND" V 9055 5222 50  0000 R CNN
+F 2 "" H 9050 5350 50  0001 C CNN
+F 3 "" H 9050 5350 50  0001 C CNN
+	1    9050 5350
+	1    0    0    -1
+$EndComp
+Wire Wire Line
+	8800 5050 8800 4950
+Wire Wire Line
+	9050 5050 9050 4950
+Wire Wire Line
+	8250 4850 8250 4950
+Connection ~ 8800 4950
+Wire Wire Line
+	8800 4950 9050 4950
+Connection ~ 9050 4950
+Wire Wire Line
+	9050 4950 9200 4950
+Wire Wire Line
+	8250 4950 8800 4950
 $EndSCHEMATC
